Commit message: updated robot name and used lower case letters for file extensions

File: motoman_bmda3_support/urdf/motoman_bmda3_macro.xacro (robot description, xacro)
@@ -13,5 +13,5 @@
       <geometry>
         <mesh
-          filename="package://motoman_bmda3_support/meshes/bmda3/visual/base_link.STL" />
+          filename="package://motoman_bmda3_support/meshes/bmda3/visual/base_link.stl" />
       </geometry>
       <material
@@ -27,5 +27,5 @@
       <geometry>
         <mesh
-          filename="package://motoman_bmda3_support/meshes/bmda3/collision/base_link.STL" />
+          filename="package://motoman_bmda3_support/meshes/bmda3/collision/base_link.stl" />
       </geometry>
     </collision>
@@ -39,5 +39,5 @@
       <geometry>
         <mesh
-          filename="package://motoman_bmda3_support/meshes/bmda3/visual/waist_link.STL" />
+          filename="package://motoman_bmda3_support/meshes/bmda3/visual/waist_link.stl" />
       </geometry>
       <material
@@ -53,5 +53,5 @@
       <geometry>
         <mesh
-          filename="package://motoman_bmda3_support/meshes/bmda3/collision/waist_link.STL" />
+          filename="package://motoman_bmda3_support/meshes/bmda3/collision/waist_link.stl" />
       </geometry>
     </collision>
@@ -65,5 +65,5 @@
       <geometry>
         <mesh
-          filename="package://motoman_bmda3_support/meshes/bmda3/visual/right_L_link.STL" />
+          filename="package://motoman_bmda3_support/meshes/bmda3/visual/right_L_link.stl" />
       </geometry>
       <material
@@ -79,5 +79,5 @@
       <geometry>
         <mesh
-          filename="package://motoman_bmda3_support/meshes/bmda3/collision/right_L_link.STL" />
+          filename="package://motoman_bmda3_support/meshes/bmda3/collision/right_L_link.stl" />
       </geometry>
     </collision>
@@ -91,5 +91,5 @@
       <geometry>
         <mesh
-          filename="package://motoman_bmda3_support/meshes/bmda3/visual/right_E_link.STL" />
+          filename="package://motoman_bmda3_support/meshes/bmda3/visual/right_E_link.stl" />
       </geometry>
       <material
@@ -105,5 +105,5 @@
       <geometry>
         <mesh
-          filename="package://motoman_bmda3_support/meshes/bmda3/collision/right_E_link.STL" />
+          filename="package://motoman_bmda3_support/meshes/bmda3/collision/right_E_link.stl" />
       </geometry>
     </collision>
@@ -117,19 +117,19 @@
       <geometry>
         <mesh
-          filename="package://motoman_bmda3_support/meshes/bmda3/visual/right_U_link.STL" />
-      </geometry>
-      <material
-        name="">
-        <color
-          rgba="0.752941176470588 0.752941176470588 0.752941176470588 1" />
-      </material>
-    </visual>
-    <collision>
-      <origin
-        xyz="0 0 0"
-        rpy="0 0 0" />
-      <geometry>
-        <mesh
-          filename="package://motoman_bmda3_support/meshes/bmda3/collision/right_U_link.STL" />
+          filename="package://motoman_bmda3_support/meshes/bmda3/visual/right_U_link.stl" />
+      </geometry>
+      <material
+        name="">
+        <color
+          rgba="0.752941176470588 0.752941176470588 0.752941176470588 1" />
+      </material>
+    </visual>
+    <collision>
+      <origin
+        xyz="0 0 0"
+        rpy="0 0 0" />
+      <geometry>
+        <mesh
+          filename="package://motoman_bmda3_support/meshes/bmda3/collision/right_U_link.stl" />
       </geometry>
     </collision>
@@ -143,19 +143,19 @@
       <geometry>
         <mesh
-          filename="package://motoman_bmda3_support/meshes/bmda3/visual/right_R_link.STL" />
-      </geometry>
-      <material
-        name="">
-        <color
-          rgba="0.752941176470588 0.752941176470588 0.752941176470588 1" />
-      </material>
-    </visual>
-    <collision>
-      <origin
-        xyz="0 0 0"
-        rpy="0 0 0" />
-      <geometry>
-        <mesh
-          filename="package://motoman_bmda3_support/meshes/bmda3/collision/right_R_link.STL" />
+          filename="package://motoman_bmda3_support/meshes/bmda3/visual/right_R_link.stl" />
+      </geometry>
+      <material
+        name="">
+        <color
+          rgba="0.752941176470588 0.752941176470588 0.752941176470588 1" />
+      </material>
+    </visual>
+    <collision>
+      <origin
+        xyz="0 0 0"
+        rpy="0 0 0" />
+      <geometry>
+        <mesh
+          filename="package://motoman_bmda3_support/meshes/bmda3/collision/right_R_link.stl" />
       </geometry>
     </collision>
@@ -169,19 +169,19 @@
       <geometry>
         <mesh
-          filename="package://motoman_bmda3_support/meshes/bmda3/visual/right_B_link.STL" />
-      </geometry>
-      <material
-        name="">
-        <color
-          rgba="0.752941176470588 0.752941176470588 0.752941176470588 1" />
-      </material>
-    </visual>
-    <collision>
-      <origin
-        xyz="0 0 0"
-        rpy="0 0 0" />
-      <geometry>
-        <mesh
-          filename="package://motoman_bmda3_support/meshes/bmda3/collision/right_B_link.STL" />
+          filename="package://motoman_bmda3_support/meshes/bmda3/visual/right_B_link.stl" />
+      </geometry>
+      <material
+        name="">
+        <color
+          rgba="0.752941176470588 0.752941176470588 0.752941176470588 1" />
+      </material>
+    </visual>
+    <collision>
+      <origin
+        xyz="0 0 0"
+        rpy="0 0 0" />
+      <geometry>
+        <mesh
+          filename="package://motoman_bmda3_support/meshes/bmda3/collision/right_B_link.stl" />
       </geometry>
     </collision>
@@ -195,19 +195,19 @@
       <geometry>
         <mesh
-          filename="package://motoman_bmda3_support/meshes/bmda3/visual/right_T_link.STL" />
-      </geometry>
-      <material
-        name="">
-        <color
-          rgba="0.752941176470588 0.752941176470588 0.752941176470588 1" />
-      </material>
-    </visual>
-    <collision>
-      <origin
-        xyz="0 0 0"
-        rpy="0 0 0" />
-      <geometry>
-        <mesh
-          filename="package://motoman_bmda3_support/meshes/bmda3/collision/right_T_link.STL" />
+          filename="package://motoman_bmda3_support/meshes/bmda3/visual/right_T_link.stl" />
+      </geometry>
+      <material
+        name="">
+        <color
+          rgba="0.752941176470588 0.752941176470588 0.752941176470588 1" />
+      </material>
+    </visual>
+    <collision>
+      <origin
+        xyz="0 0 0"
+        rpy="0 0 0" />
+      <geometry>
+        <mesh
+          filename="package://motoman_bmda3_support/meshes/bmda3/collision/right_T_link.stl" />
       </geometry>
     </collision>
@@ -221,19 +221,19 @@
       <geometry>
         <mesh
-          filename="package://motoman_bmda3_support/meshes/bmda3/visual/right_tool_0.STL" />
-      </geometry>
-      <material
-        name="">
-        <color
-          rgba="0.752941176470588 0.752941176470588 0.752941176470588 1" />
-      </material>
-    </visual>
-    <collision>
-      <origin
-        xyz="0 0 0"
-        rpy="0 0 0" />
-      <geometry>
-        <mesh
-          filename="package://motoman_bmda3_support/meshes/bmda3/collision/right_tool_0.STL" />
+          filename="package://motoman_bmda3_support/meshes/bmda3/visual/right_tool_0.stl" />
+      </geometry>
+      <material
+        name="">
+        <color
+          rgba="0.752941176470588 0.752941176470588 0.752941176470588 1" />
+      </material>
+    </visual>
+    <collision>
+      <origin
+        xyz="0 0 0"
+        rpy="0 0 0" />
+      <geometry>
+        <mesh
+          filename="package://motoman_bmda3_support/meshes/bmda3/collision/right_tool_0.stl" />
       </geometry>
     </collision>
@@ -247,19 +247,19 @@
       <geometry>
         <mesh
-          filename="package://motoman_bmda3_support/meshes/bmda3/visual/left_L_link.STL" />
-      </geometry>
-      <material
-        name="">
-        <color
-          rgba="0.752941176470588 0.752941176470588 0.752941176470588 1" />
-      </material>
-    </visual>
-    <collision>
-      <origin
-        xyz="0 0 0"
-        rpy="0 0 0" />
-      <geometry>
-        <mesh
-          filename="package://motoman_bmda3_support/meshes/bmda3/collision/left_L_link.STL" />
+          filename="package://motoman_bmda3_support/meshes/bmda3/visual/left_L_link.stl" />
+      </geometry>
+      <material
+        name="">
+        <color
+          rgba="0.752941176470588 0.752941176470588 0.752941176470588 1" />
+      </material>
+    </visual>
+    <collision>
+      <origin
+        xyz="0 0 0"
+        rpy="0 0 0" />
+      <geometry>
+        <mesh
+          filename="package://motoman_bmda3_support/meshes/bmda3/collision/left_L_link.stl" />
       </geometry>
     </collision>
@@ -273,19 +273,19 @@
       <geometry>
         <mesh
-          filename="package://motoman_bmda3_support/meshes/bmda3/visual/left_E_link.STL" />
-      </geometry>
-      <material
-        name="">
-        <color
-          rgba="0.752941176470588 0.752941176470588 0.752941176470588 1" />
-      </material>
-    </visual>
-    <collision>
-      <origin
-        xyz="0 0 0"
-        rpy="0 0 0" />
-      <geometry>
-        <mesh
-          filename="package://motoman_bmda3_support/meshes/bmda3/collision/left_E_link.STL" />
+          filename="package://motoman_bmda3_support/meshes/bmda3/visual/left_E_link.stl" />
+      </geometry>
+      <material
+        name="">
+        <color
+          rgba="0.752941176470588 0.752941176470588 0.752941176470588 1" />
+      </material>
+    </visual>
+    <collision>
+      <origin
+        xyz="0 0 0"
+        rpy="0 0 0" />
+      <geometry>
+        <mesh
+          filename="package://motoman_bmda3_support/meshes/bmda3/collision/left_E_link.stl" />
       </geometry>
     </collision>
@@ -299,19 +299,19 @@
       <geometry>
         <mesh
-          filename="package://motoman_bmda3_support/meshes/bmda3/visual/left_U_link.STL" />
-      </geometry>
-      <material
-        name="">
-        <color
-          rgba="0.752941176470588 0.752941176470588 0.752941176470588 1" />
-      </material>
-    </visual>
-    <collision>
-      <origin
-        xyz="0 0 0"
-        rpy="0 0 0" />
-      <geometry>
-        <mesh
-          filename="package://motoman_bmda3_support/meshes/bmda3/collision/left_U_link.STL" />
+          filename="package://motoman_bmda3_support/meshes/bmda3/visual/left_U_link.stl" />
+      </geometry>
+      <material
+        name="">
+        <color
+          rgba="0.752941176470588 0.752941176470588 0.752941176470588 1" />
+      </material>
+    </visual>
+    <collision>
+      <origin
+        xyz="0 0 0"
+        rpy="0 0 0" />
+      <geometry>
+        <mesh
+          filename="package://motoman_bmda3_support/meshes/bmda3/collision/left_U_link.stl" />
       </geometry>
     </collision>
@@ -325,19 +325,19 @@
       <geometry>
         <mesh
-          filename="package://motoman_bmda3_support/meshes/bmda3/visual/left_R_link.STL" />
-      </geometry>
-      <material
-        name="">
-        <color
-          rgba="0.752941176470588 0.752941176470588 0.752941176470588 1" />
-      </material>
-    </visual>
-    <collision>
-      <origin
-        xyz="0 0 0"
-        rpy="0 0 0" />
-      <geometry>
-        <mesh
-          filename="package://motoman_bmda3_support/meshes/bmda3/collision/left_R_link.STL" />
+          filename="package://motoman_bmda3_support/meshes/bmda3/visual/left_R_link.stl" />
+      </geometry>
+      <material
+        name="">
+        <color
+          rgba="0.752941176470588 0.752941176470588 0.752941176470588 1" />
+      </material>
+    </visual>
+    <collision>
+      <origin
+        xyz="0 0 0"
+        rpy="0 0 0" />
+      <geometry>
+        <mesh
+          filename="package://motoman_bmda3_support/meshes/bmda3/collision/left_R_link.stl" />
       </geometry>
     </collision>
@@ -351,19 +351,19 @@
       <geometry>
         <mesh
-          filename="package://motoman_bmda3_support/meshes/bmda3/visual/left_B_link.STL" />
-      </geometry>
-      <material
-        name="">
-        <color
-          rgba="0.752941176470588 0.752941176470588 0.752941176470588 1" />
-      </material>
-    </visual>
-    <collision>
-      <origin
-        xyz="0 0 0"
-        rpy="0 0 0" />
-      <geometry>
-        <mesh
-          filename="package://motoman_bmda3_support/meshes/bmda3/collision/left_B_link.STL" />
+          filename="package://motoman_bmda3_support/meshes/bmda3/visual/left_B_link.stl" />
+      </geometry>
+      <material
+        name="">
+        <color
+          rgba="0.752941176470588 0.752941176470588 0.752941176470588 1" />
+      </material>
+    </visual>
+    <collision>
+      <origin
+        xyz="0 0 0"
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