Commit message: Changed naming convention for links and joints. Updated names of mesh files.

File: motoman_bmda3_support/urdf/motoman_bmda3.urdf (robot description, URDF)
Before this commit: robot motoman_bmda3, 17 links, 16 joints
Links:
- removed link left_B_link
- removed link left_E_link
- removed link left_L_link
- removed link left_R_link
- removed link left_T_link
- removed link left_U_link
- removed link right_B_link
- removed link right_E_link
- removed link right_L_link
- removed link right_R_link
- removed link right_T_link
- removed link right_U_link
- removed link world
- added link base; collision mesh filename=package://motoman_bmda3_support/meshes/bmda3/collision/base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; visual mesh filename=package://motoman_bmda3_support/meshes/bmda3/visual/base.stl
- added link left_link_B; collision mesh filename=package://motoman_bmda3_support/meshes/bmda3/collision/left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; visual mesh filename=package://motoman_bmda3_support/meshes/bmda3/visual/left_li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
- added link left_link_E; collision mesh filename=package://motoman_bmda3_support/meshes/bmda3/collision/left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; visual mesh filename=package://motoman_bmda3_support/meshes/bmda3/visual/left_li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
- added link left_link_L; collision mesh filename=package://motoman_bmda3_support/meshes/bmda3/collision/left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; visual mesh filename=package://motoman_bmda3_support/meshes/bmda3/visual/left_li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
- added link left_link_R; collision mesh filename=package://motoman_bmda3_support/meshes/bmda3/collision/left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; visual mesh filename=package://motoman_bmda3_support/meshes/bmda3/visual/left_li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
- added link left_link_T; collision mesh filename=package://motoman_bmda3_support/meshes/bmda3/collision/left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; visual mesh filename=package://motoman_bmda3_support/meshes/bmda3/visual/left_li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
- added link left_link_U; collision mesh filename=package://motoman_bmda3_support/meshes/bmda3/collision/left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; visual mesh filename=package://motoman_bmda3_support/meshes/bmda3/visual/left_li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
- added link right_link_B; collision mesh filename=package://motoman_bmda3_support/meshes/bmda3/collision/righ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; visual mesh filename=package://motoman_bmda3_support/meshes/bmda3/visual/right_l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
- added link right_link_E; collision mesh filename=package://motoman_bmda3_support/meshes/bmda3/collision/righ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; visual mesh filename=package://motoman_bmda3_support/meshes/bmda3/visual/right_l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
- added link right_link_L; collision mesh filename=package://motoman_bmda3_support/meshes/bmda3/collision/righ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; visual mesh filename=package://motoman_bmda3_support/meshes/bmda3/visual/right_l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
- added link right_link_R; collision mesh filename=package://motoman_bmda3_support/meshes/bmda3/collision/righ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; visual mesh filename=package://motoman_bmda3_support/meshes/bmda3/visual/right_l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
- added link right_link_T; collision mesh filename=package://motoman_bmda3_support/meshes/bmda3/collision/righ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; visual mesh filename=package://motoman_bmda3_support/meshes/bmda3/visual/right_l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
- added link right_link_U; collision mesh filename=package://motoman_bmda3_support/meshes/bmda3/collision/righ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; visual mesh filename=package://motoman_bmda3_support/meshes/bmda3/visual/right_l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
- link base_link: geometry 
Joints:
- removed joint left_B_axis
- removed joint left_E_axis
- removed joint left_L_axis
- removed joint left_R_axis
- removed joint left_S_axis
- removed joint left_T_axis
- removed joint left_U_axis
- removed joint right_B_axis
- removed joint right_E_axis
- removed joint right_L_axis
- removed joint right_R_axis
- removed joint right_S_axis
- removed joint right_T_axis
- removed joint right_U_axis
- removed joint waist_axis
- removed joint world-base
- added joint base_link-base: type fixed, parent base_link, child base, origin xyz=0 0 0 rpy=0 0 0
- added joint left_joint_B: type revolute, parent left_link_B, child left_link_T, origin xyz=0 0 0 rpy=0 0 0, axis 0 0 1, limit lower=-1.9198 upper=1.9198 effort=0 velocity=3.49
- added joint left_joint_E: type revolute, parent left_link_E, child left_link_U, origin xyz=0 0.23549999999989 0 rpy=0 0 0, axis 0 1 0, limit lower=-2.966 upper=2.966 effort=0 velocity=2.97
- added joint left_joint_L: type revolute, parent left_link_L, child left_link_E, origin xyz=0 0.151 0 rpy=0 0 0, axis 0 0 -1, limit lower=-1.745 upper=1.745 effort=0 velocity=2.62
- added joint left_joint_R: type revolute, parent left_link_R, child left_link_B, origin xyz=0.35997 0.05 0 rpy=0 0 0, axis -1 0 0, limit lower=-3.1415 upper=3.1415 effort=0 velocity=3.49
- added joint left_joint_S: type revolute, parent waist_link, child left_link_L, origin xyz=0.15003 0.099 0.1295 rpy=0 0 0, axis 0 1 0, limit lower=-1.57 upper=3.1415 effort=0 velocity=2.97
- added joint left_joint_T: type revolute, parent left_link_T, child left_tool_0, origin xyz=0.138 0 0 rpy=0 0 0, axis -1 0 0, limit lower=-4.712 upper=4.712 effort=0 velocity=6.11
- added joint left_joint_U: type revolute, parent left_link_U, child left_link_R, origin xyz=0.065 0.1445 0 rpy=0 0 0, axis 0 0 1, limit lower=-1.396 upper=0.7504 effort=0 velocity=2.97
- added joint right_joint_B: type revolute, parent right_link_B, child right_link_T, origin xyz=0 0 0 rpy=0 0 0, axis 0 0 -1, limit lower=-1.9198 upper=1.9198 effort=0 velocity=3.49
- added joint right_joint_E: type revolute, parent right_link_E, child right_link_U, origin xyz=0 -0.23549999999989 0 rpy=0 0 0, axis 0 1 0, limit lower=-2.966 upper=2.966 effort=0 velocity=2.97
- added joint right_joint_L: type revolute, parent right_link_L, child right_link_E, origin xyz=0 -0.151 0 rpy=0 0 0, axis 0 0 1, limit lower=-1.745 upper=1.745 effort=0 velocity=2.62
- added joint right_joint_R: type revolute, parent right_link_R, child right_link_B, origin xyz=0.35997 -0.05 0 rpy=0 0 0, axis 1 0 0, limit lower=-3.1415 upper=3.1415 effort=0 velocity=3.49
- added joint right_joint_S: type revolute, parent waist_link, child right_link_L, origin xyz=0.15002 -0.099 0.12951 rpy=0 0 0, axis 0 1 0, limit lower=-1.57 upper=3.14 effort=0 velocity=2.97
- added joint right_joint_T: type revolute, parent right_link_T, child right_tool_0, origin xyz=0.138 0 0 rpy=0 0 0, axis 1 0 0, limit lower=-4.712 upper=4.712 effort=0 velocity=6.11
- added joint right_joint_U: type revolute, parent right_link_U, child right_link_R, origin xyz=0.065002 -0.1445 0 rpy=0 0 0, axis 0 0 -1, limit lower=-1.396 upper=0.7504 effort=0 velocity=2.97
- added joint waist: type revolute, parent base, child waist_link, origin xyz=0 0 0.3305 rpy=0 0 0, axis 0 0 1, limit lower=-3.14 upper=3.14 effort=0 velocity=2.27

File: motoman_bmda3_support/urdf/motoman_bmda3_macro.xacro (robot description, xacro)
@@ -3,8 +3,8 @@
     <xacro:macro name="motoman_bmda3" params="prefix">
 		<!-- link list -->
-		<link name="world">
+		<link name="base_link">
     		<origin xyz="0 0 0" rpy="0 0 0"/>
   	</link>
-		<link name="${prefix}base_link">
+		<link name="${prefix}base">
       <visual>
       <origin
@@ -13,5 +13,5 @@
       <geometry>
         <mesh
-          filename="package://motoman_bmda3_support/meshes/bmda3/visual/base_link.stl" />
+          filename="package://motoman_bmda3_support/meshes/bmda3/visual/base.stl" />
       </geometry>
       <material
@@ -27,5 +27,5 @@
       <geometry>
         <mesh
-          filename="package://motoman_bmda3_support/meshes/bmda3/collision/base_link.stl" />
+          filename="package://motoman_bmda3_support/meshes/bmda3/collision/base.stl" />
       </geometry>
     </collision>
@@ -58,12 +58,12 @@
   </link>
   <link
-    name="${prefix}right_L_link">
-    <visual>
-      <origin
-        xyz="0 0 0"
-        rpy="0 0 0" />
-      <geometry>
-        <mesh
-          filename="package://motoman_bmda3_support/meshes/bmda3/visual/right_L_link.stl" />
+    name="${prefix}right_link_L">
+    <visual>
+      <origin
+        xyz="0 0 0"
+        rpy="0 0 0" />
+      <geometry>
+        <mesh
+          filename="package://motoman_bmda3_support/meshes/bmda3/visual/right_link_L.stl" />
       </geometry>
       <material
@@ -79,17 +79,17 @@
       <geometry>
         <mesh
-          filename="package://motoman_bmda3_support/meshes/bmda3/collision/right_L_link.stl" />
-      </geometry>
-    </collision>
-  </link>
-  <link
-    name="${prefix}right_E_link">
-    <visual>
-      <origin
-        xyz="0 0 0"
-        rpy="0 0 0" />
-      <geometry>
-        <mesh
-          filename="package://motoman_bmda3_support/meshes/bmda3/visual/right_E_link.stl" />
+          filename="package://motoman_bmda3_support/meshes/bmda3/collision/right_link_L.stl" />
+      </geometry>
+    </collision>
+  </link>
+  <link
+    name="${prefix}right_link_E">
+    <visual>
+      <origin
+        xyz="0 0 0"
+        rpy="0 0 0" />
+      <geometry>
+        <mesh
+          filename="package://motoman_bmda3_support/meshes/bmda3/visual/right_link_E.stl" />
       </geometry>
       <material
@@ -105,10 +105,10 @@
       <geometry>
         <mesh
-          filename="package://motoman_bmda3_support/meshes/bmda3/collision/right_E_link.stl" />
-      </geometry>
-    </collision>
-  </link>
-  <link
-    name="${prefix}right_U_link">
+          filename="package://motoman_bmda3_support/meshes/bmda3/collision/right_link_E.stl" />
+      </geometry>
+    </collision>
+  </link>
+  <link
+    name="${prefix}right_link_U">
      <visual>
       <origin
@@ -117,97 +117,97 @@
       <geometry>
         <mesh
-          filename="package://motoman_bmda3_support/meshes/bmda3/visual/right_U_link.stl" />
-      </geometry>
-      <material
-        name="">
-        <color
-          rgba="0.752941176470588 0.752941176470588 0.752941176470588 1" />
-      </material>
-    </visual>
-    <collision>
-      <origin
-        xyz="0 0 0"
-        rpy="0 0 0" />
-      <geometry>
-        <mesh
-          filename="package://motoman_bmda3_support/meshes/bmda3/collision/right_U_link.stl" />
-      </geometry>
-    </collision>
-  </link>
-  <link
-    name="${prefix}right_R_link">
-    <visual>
-      <origin
-        xyz="0 0 0"
-        rpy="0 0 0" />
-      <geometry>
-        <mesh
-          filename="package://motoman_bmda3_support/meshes/bmda3/visual/right_R_link.stl" />
-      </geometry>
-      <material
-        name="">
-        <color
-          rgba="0.752941176470588 0.752941176470588 0.752941176470588 1" />
-      </material>
-    </visual>
-    <collision>
-      <origin
-        xyz="0 0 0"
-        rpy="0 0 0" />
-      <geometry>
-        <mesh
-          filename="package://motoman_bmda3_support/meshes/bmda3/collision/right_R_link.stl" />
-      </geometry>
-    </collision>
-  </link>
-  <link
-    name="${prefix}right_B_link">
-    <visual>
-      <origin
-        xyz="0 0 0"
-        rpy="0 0 0" />
-      <geometry>
-        <mesh
-          filename="package://motoman_bmda3_support/meshes/bmda3/visual/right_B_link.stl" />
-      </geometry>
-      <material
-        name="">
-        <color
-          rgba="0.752941176470588 0.752941176470588 0.752941176470588 1" />
-      </material>
-    </visual>
-    <collision>
-      <origin
-        xyz="0 0 0"
-        rpy="0 0 0" />
-      <geometry>
-        <mesh
-          filename="package://motoman_bmda3_support/meshes/bmda3/collision/right_B_link.stl" />
-      </geometry>
-    </collision>
-  </link>
-  <link
-    name="${prefix}right_T_link">
-    <visual>
-      <origin
-        xyz="0 0 0"
-        rpy="0 0 0" />
-      <geometry>
-        <mesh
-          filename="package://motoman_bmda3_support/meshes/bmda3/visual/right_T_link.stl" />
-      </geometry>
-      <material
-        name="">
-        <color
-          rgba="0.752941176470588 0.752941176470588 0.752941176470588 1" />
-      </material>
-    </visual>
-    <collision>
-      <origin
-        xyz="0 0 0"
-        rpy="0 0 0" />
-      <geometry>
-        <mesh
-          filename="package://motoman_bmda3_support/meshes/bmda3/collision/right_T_link.stl" />
+          filename="package://motoman_bmda3_support/meshes/bmda3/visual/right_link_U.stl" />
+      </geometry>
+      <material
+        name="">
+        <color
+          rgba="0.752941176470588 0.752941176470588 0.752941176470588 1" />
+      </material>
+    </visual>
+    <collision>
+      <origin
+        xyz="0 0 0"
+        rpy="0 0 0" />
+      <geometry>
+        <mesh
+          filename="package://motoman_bmda3_support/meshes/bmda3/collision/right_link_U.stl" />
+      </geometry>
+    </collision>
+  </link>
+  <link
+    name="${prefix}right_link_R">
+    <visual>
+      <origin
+        xyz="0 0 0"
+        rpy="0 0 0" />
+      <geometry>
+        <mesh
+          filename="package://motoman_bmda3_support/meshes/bmda3/visual/right_link_R.stl" />
+      </geometry>
+      <material
+        name="">
+        <color
+          rgba="0.752941176470588 0.752941176470588 0.752941176470588 1" />
+      </material>
+    </visual>
+    <collision>
+      <origin
+        xyz="0 0 0"
+        rpy="0 0 0" />
+      <geometry>
+        <mesh
+          filename="package://motoman_bmda3_support/meshes/bmda3/collision/right_link_R.stl" />
+      </geometry>
+    </collision>
+  </link>
+  <link
+    name="${prefix}right_link_B">
+    <visual>
+      <origin
+        xyz="0 0 0"
+        rpy="0 0 0" />
+      <geometry>
+        <mesh
+          filename="package://motoman_bmda3_support/meshes/bmda3/visual/right_link_B.stl" />
+      </geometry>
+      <material
+        name="">
+        <color
+          rgba="0.752941176470588 0.752941176470588 0.752941176470588 1" />
+      </material>
+    </visual>
+    <collision>
+      <origin
+        xyz="0 0 0"
+        rpy="0 0 0" />
+      <geometry>
+        <mesh
+          filename="package://motoman_bmda3_support/meshes/bmda3/collision/right_link_B.stl" />
+      </geometry>
+    </collision>
+  </link>
+  <link
+    name="${prefix}right_link_T">
+    <visual>
+      <origin
+        xyz="0 0 0"
+        rpy="0 0 0" />
+      <geometry>
+        <mesh
+          filename="package://motoman_bmda3_support/meshes/bmda3/visual/right_link_T.stl" />
+      </geometry>
+      <material
+        name="">
+        <color
+          rgba="0.752941176470588 0.752941176470588 0.752941176470588 1" />
+      </material>
+    </visual>
+    <collision>
+      <origin
+        xyz="0 0 0"
+        rpy="0 0 0" />
+      <geometry>
+        <mesh
+          filename="package://motoman_bmda3_support/meshes/bmda3/collision/right_link_T.stl" />
       </geometry>
     </collision>
@@ -240,156 +240,156 @@
   </link>
   <link
-    name="${prefix}left_L_link">
-    <visual>
-      <origin
-        xyz="0 0 0"
-        rpy="0 0 0" />
-      <geometry>
-        <mesh
-          filename="package://motoman_bmda3_support/meshes/bmda3/visual/left_L_link.stl" />
-      </geometry>
-      <material
-        name="">
-        <color
-          rgba="0.752941176470588 0.752941176470588 0.752941176470588 1" />
-      </material>
-    </visual>
-    <collision>
-      <origin
-        xyz="0 0 0"
-        rpy="0 0 0" />
-      <geometry>
-        <mesh
-          filename="package://motoman_bmda3_support/meshes/bmda3/collision/left_L_link.stl" />
-      </geometry>
-    </collision>
-  </link>
-  <link
-    name="${prefix}left_E_link">
-    <visual>
-      <origin
-        xyz="0 0 0"
-        rpy="0 0 0" />
-      <geometry>
-        <mesh
-          filename="package://motoman_bmda3_support/meshes/bmda3/visual/left_E_link.stl" />
-      </geometry>
-      <material
-        name="">
-        <color
-          rgba="0.752941176470588 0.752941176470588 0.752941176470588 1" />
-      </material>
-    </visual>
-    <collision>
-      <origin
-        xyz="0 0 0"
-        rpy="0 0 0" />
-      <geometry>
-        <mesh
-          filename="package://motoman_bmda3_support/meshes/bmda3/collision/left_E_link.stl" />
-      </geometry>
-    </collision>
-  </link>
-  <link
-    name="${prefix}left_U_link">
-    <visual>
-      <origin
-        xyz="0 0 0"
-        rpy="0 0 0" />
-      <geometry>
-        <mesh
-          filename="package://motoman_bmda3_support/meshes/bmda3/visual/left_U_link.stl" />
-      </geometry>
-      <material
-        name="">
-        <color
-          rgba="0.752941176470588 0.752941176470588 0.752941176470588 1" />
-      </material>
-    </visual>
-    <collision>
-      <origin
-        xyz="0 0 0"
-        rpy="0 0 0" />
-      <geometry>
-        <mesh
-          filename="package://motoman_bmda3_support/meshes/bmda3/collision/left_U_link.stl" />
-      </geometry>
-    </collision>
-  </link>
-  <link
-    name="${prefix}left_R_link">
-    <visual>
-      <origin
-        xyz="0 0 0"
-        rpy="0 0 0" />
-      <geometry>
-        <mesh
-          filename="package://motoman_bmda3_support/meshes/bmda3/visual/left_R_link.stl" />
-      </geometry>
-      <material
-        name="">
-        <color
-          rgba="0.752941176470588 0.752941176470588 0.752941176470588 1" />
-      </material>
-    </visual>
-    <collision>
-      <origin
-        xyz="0 0 0"
-        rpy="0 0 0" />
-      <geometry>
-        <mesh
-          filename="package://motoman_bmda3_support/meshes/bmda3/collision/left_R_link.stl" />
-      </geometry>
-    </collision>
-  </link>
-  <link
-    name="${prefix}left_B_link">
-    <visual>
-      <origin
-        xyz="0 0 0"
-        rpy="0 0 0" />
-      <geometry>
-        <mesh
-          filename="package://motoman_bmda3_support/meshes/bmda3/visual/left_B_link.stl" />
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