Commit message: Renamed "waist" to "torso", created torso_joint_b1 and torso_joint_b2.

File: motoman_bmda3_support/urdf/bmda3.urdf (robot description, URDF)
Before this commit: robot motoman_bmda3, 17 links, 16 joints
Links:
- removed link waist_link
- added link torso_link_b1; collision mesh filename=package://motoman_bmda3_support/meshes/bmda3/collision/tors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; visual mesh filename=package://motoman_bmda3_support/meshes/bmda3/visual/torso_l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
- added link torso_link_b2; collision mesh filename=package://motoman_bmda3_support/meshes/bmda3/collision/tors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; visual mesh filename=package://motoman_bmda3_support/meshes/bmda3/visual/torso_l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
Joints:
- removed joint waist
- added joint torso_joint_b1: type revolute, parent base, child torso_link_b1, origin xyz=0 0 0.3305 rpy=0 0 0, axis 0 0 1, limit lower=-3.1415 upper=3.1415 effort=0 velocity=2.27
- added joint torso_joint_b2: type revolute, parent base, child torso_link_b2, origin xyz=0 0 0.3305 rpy=0 0 0, axis 0 0 1, limit lower=-3.1415 upper=3.1415 effort=0 velocity=2.27
- joint left_joint_s: parent waist_link -> torso_link_b1
- joint right_joint_s: parent waist_link -> torso_link_b1

File: motoman_bmda3_support/urdf/bmda3_macro.xacro (robot description, xacro)
@@ -32,12 +32,12 @@
   </link>
   <link
-    name="${prefix}waist_link">
-    <visual>
-      <origin
-        xyz="0 0 0"
-        rpy="0 0 0" />
-      <geometry>
-        <mesh
-          filename="package://motoman_bmda3_support/meshes/bmda3/visual/waist_link.stl" />
+    name="${prefix}torso_link_b1">
+    <visual>
+      <origin
+        xyz="0 0 0"
+        rpy="0 0 0" />
+      <geometry>
+        <mesh
+          filename="package://motoman_bmda3_support/meshes/bmda3/visual/torso_link.stl" />
       </geometry>
       <material
@@ -53,5 +53,5 @@
       <geometry>
         <mesh
-          filename="package://motoman_bmda3_support/meshes/bmda3/collision/waist_link.stl" />
+          filename="package://motoman_bmda3_support/meshes/bmda3/collision/torso_link.stl" />
       </geometry>
     </collision>
@@ -214,4 +214,31 @@
   </link>
   <link name="${prefix}right_tool0" />
+  <!-- Note that the redundant torso link b2 is introduced to match the phantom joint in the controller -->
+  <link
+    name="${prefix}torso_link_b2">
+    <visual>
+      <origin
+        xyz="0 0 0"
+        rpy="0 0 0" />
+      <geometry>
+        <mesh
+          filename="package://motoman_bmda3_support/meshes/bmda3/visual/torso_link.stl" />
+      </geometry>
+      <material
+        name="">
+        <color
+          rgba="0.75294 0.75294 0.75294 1" />
+      </material>
+    </visual>
+    <collision>
+      <origin
+        xyz="0 0 0"
+        rpy="0 0 0" />
+      <geometry>
+        <mesh
+          filename="package://motoman_bmda3_support/meshes/bmda3/collision/torso_link.stl" />
+      </geometry>
+    </collision>
+  </link>
   <link
     name="${prefix}left_link_l">
@@ -378,7 +405,7 @@
    	<child link="${prefix}base"/>
   	</joint>
-    <joint name="${prefix}waist" type="revolute">
+    <joint name="${prefix}torso_joint_b1" type="revolute">
           <parent link="${prefix}base" />
-          <child  link="${prefix}waist_link" />
+          <child  link="${prefix}torso_link_b1" />
           <origin xyz="0 0 0.3305" rpy="0 0 0" />
           <axis xyz="0 0 1" />
@@ -386,5 +413,5 @@
     </joint>
     <joint name="${prefix}right_joint_s" type="revolute">
-          <parent link="${prefix}waist_link" />
+          <parent link="${prefix}torso_link_b1" />
           <child link="${prefix}right_link_l" />
           <origin xyz="0.15002 -0.099 0.12951" rpy="0 0 0" />
@@ -434,6 +461,14 @@
           <limit lower="-4.712" upper="4.712" effort="0" velocity="6.11" />
     </joint>
+    <!-- Note that the redundant torso joint b2 is introduced to match the phantom joint in the controller -->
+    <joint name="${prefix}torso_joint_b2" type="revolute">
+          <parent link="${prefix}base" />
+          <child  link="${prefix}torso_link_b2" />
+          <origin xyz="0 0 0.3305" rpy="0 0 0" />
+          <axis xyz="0 0 1" />
+          <limit lower="-3.1415" upper="3.1415" effort="0" velocity="2.27" />
+    </joint>
     <joint name="${prefix}left_joint_s" type="revolute">
-          <parent link="${prefix}waist_link" />
+          <parent link="${prefix}torso_link_b1" />
           <child link="${prefix}left_link_l" />
           <origin xyz="0.15003 0.099 0.1295" rpy="0 0 0" />

File: motoman_bmda3_support/urdf/bmda3_w_effs.urdf (robot description, URDF)
Before this commit: robot motoman_bmda3_w_effs, 19 links, 18 joints
Links:
- removed link waist_link
- added link torso_link_b1; collision mesh filename=package://motoman_bmda3_support/meshes/bmda3/collision/tors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; visual mesh filename=package://motoman_bmda3_support/meshes/bmda3/visual/torso_l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
- added link torso_link_b2; collision mesh filename=package://motoman_bmda3_support/meshes/bmda3/collision/tors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; visual mesh filename=package://motoman_bmda3_support/meshes/bmda3/visual/torso_l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
Joints:
- removed joint waist
- added joint torso_joint_b1: type revolute, parent base, child torso_link_b1, origin xyz=0 0 0.3305 rpy=0 0 0, axis 0 0 1, limit lower=-3.1415 upper=3.1415 effort=0 velocity=2.27
- added joint torso_joint_b2: type revolute, parent base, child torso_link_b2, origin xyz=0 0 0.3305 rpy=0 0 0, axis 0 0 1, limit lower=-3.1415 upper=3.1415 effort=0 velocity=2.27
- joint left_joint_s: parent waist_link -> torso_link_b1
- joint right_joint_s: parent waist_link -> torso_link_b1

Commit message: new branch for single bmda3 config files

File: motoman_bmda3_support/urdf/bmda3.urdf (robot description, URDF)
Before this commit: robot motoman_bmda3, 18 links, 17 joints
Links:
- added link left_eff; collision mesh filename=package://motoman_bmda3_support/meshes/bmda3/collision/eff.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; visual mesh filename=package://motoman_bmda3_support/meshes/bmda3/visual/eff.stl
- added link right_eff; collision mesh filename=package://motoman_bmda3_support/meshes/bmda3/collision/eff.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; visual mesh filename=package://motoman_bmda3_support/meshes/bmda3/visual/eff.stl
Joints:
- removed joint left_joint_b
- removed joint left_joint_e
- removed joint left_joint_l
- removed joint left_joint_r
- removed joint left_joint_s
- removed joint left_joint_t
- removed joint left_joint_u
- removed joint right_joint_b
- removed joint right_joint_e
- removed joint right_joint_l
- removed joint right_joint_r
- removed joint right_joint_s
- removed joint right_joint_t
- removed joint right_joint_u
- added joint left_eff: type fixed, parent left_tool0, child left_eff, origin xyz=0 0 0 rpy=0 0 0, axis 0 0 1
- added joint left_joint_1_s: type revolute, parent torso_link_b1, child left_link_l, origin xyz=0.15003 0.099 0.1295 rpy=0 0 0, axis 0 1 0, limit lower=-1.570 upper=3.1415 effort=0 velocity=2.97
- added joint left_joint_2_l: type revolute, parent left_link_l, child left_link_e, origin xyz=0 0.151 0 rpy=0 0 0, axis 0 0 -1, limit lower=-1.745 upper=1.745 effort=0 velocity=2.62
- added joint left_joint_3_e: type revolute, parent left_link_e, child left_link_u, origin xyz=0 0.23549999999989 0 rpy=0 0 0, axis 0 1 0, limit lower=-2.966 upper=2.966 effort=0 velocity=2.97
- added joint left_joint_4_u: type revolute, parent left_link_u, child left_link_r, origin xyz=0.065 0.1445 0 rpy=0 0 0, axis 0 0 1, limit lower=-1.396 upper=0.7504 effort=0 velocity=2.97
- added joint left_joint_5_r: type revolute, parent left_link_r, child left_link_b, origin xyz=0.35997 0.05 0 rpy=0 0 0, axis -1 0 0, limit lower=-3.1415 upper=3.1415 effort=0 velocity=3.49
- added joint left_joint_6_b: type revolute, parent left_link_b, child left_link_t, origin xyz=0 0 0 rpy=0 0 0, axis 0 0 1, limit lower=-1.9198 upper=1.9198 effort=0 velocity=3.49
- added joint left_joint_7_t: type revolute, parent left_link_t, child left_tool0, origin xyz=0.138 0 0 rpy=0 0 0, axis -1 0 0, limit lower=-4.712 upper=4.712 effort=0 velocity=6.11
- added joint right_eff: type fixed, parent right_tool0, child right_eff, origin xyz=0 0 0 rpy=0 0 0, axis 0 0 1
- added joint right_joint_1_s: type revolute, parent torso_link_b1, child right_link_l, origin xyz=0.15002 -0.099 0.12951 rpy=0 0 0, axis 0 1 0, limit lower=-1.570 upper=3.1415 effort=0 velocity=2.97
- added joint right_joint_2_l: type revolute, parent right_link_l, child right_link_e, origin xyz=0 -0.151 0 rpy=0 0 0, axis 0 0 1, limit lower=-1.745 upper=1.745 effort=0 velocity=2.62
- added joint right_joint_3_e: type revolute, parent right_link_e, child right_link_u, origin xyz=0 -0.23549999999989 0 rpy=0 0 0, axis 0 1 0, limit lower=-2.966 upper=2.966 effort=0 velocity=2.97
- added joint right_joint_4_u: type revolute, parent right_link_u, child right_link_r, origin xyz=0.065002 -0.1445 0 rpy=0 0 0, axis 0 0 -1, limit lower=-1.396 upper=0.7504 effort=0 velocity=2.97
- added joint right_joint_5_r: type revolute, parent right_link_r, child right_link_b, origin xyz=0.35997 -0.05 0 rpy=0 0 0, axis 1 0 0, limit lower=-3.1415 upper=3.1415 effort=0 velocity=3.49
- added joint right_joint_6_b: type revolute, parent right_link_b, child right_link_t, origin xyz=0 0 0 rpy=0 0 0, axis 0 0 -1, limit lower=-1.9198 upper=1.9198 effort=0 velocity=3.49
- added joint right_joint_7_t: type revolute, parent right_link_t, child right_tool0, origin xyz=0.138 0 0 rpy=0 0 0, axis 1 0 0, limit lower=-4.712 upper=4.712 effort=0 velocity=6.11

File: motoman_bmda3_support/urdf/bmda3.xacro (robot description, xacro)
@@ -1,5 +1,20 @@
 <?xml version="1.0" ?>
 <robot name="motoman_bmda3" xmlns:xacro="http://ros.org/wiki/xacro">
+	<xacro:include filename="$(find motoman_bmda3_support)/urdf/bmda3_eff_macro.xacro" />
 	<xacro:include filename="$(find motoman_bmda3_support)/urdf/bmda3_macro.xacro" />
 	<xacro:bmda3 prefix=""/>
+        <xacro:bmda3_eff prefix="right_"/>
+        <xacro:bmda3_eff prefix="left_"/>
+	<joint name="left_eff" type="fixed" >
+          <parent link="left_tool0" />
+          <child link="left_eff" />
+          <origin xyz="0 0 0" rpy="0 0 0" />
+          <axis xyz="0 0 1" />
+        </joint>
+       <joint name="right_eff" type="fixed">
+          <parent link="right_tool0" />
+          <child link="right_eff" />
+          <origin xyz="0 0 0" rpy="0 0 0" />
+          <axis xyz="0 0 1" />
+       </joint>
 </robot>

File: motoman_bmda3_support/urdf/bmda3_macro.xacro (robot description, xacro)
@@ -412,5 +412,5 @@
           <limit lower="-3.1415" upper="3.1415" effort="0" velocity="2.27" />
     </joint>
-    <joint name="${prefix}right_joint_s" type="revolute">
+    <joint name="${prefix}right_joint_1_s" type="revolute">
           <parent link="${prefix}torso_link_b1" />
           <child link="${prefix}right_link_l" />
@@ -419,5 +419,5 @@
           <limit lower="-1.570" upper="3.1415" effort="0" velocity="2.97" />
     </joint>
-    <joint name="${prefix}right_joint_l" type="revolute">
+    <joint name="${prefix}right_joint_2_l" type="revolute">
           <parent link="${prefix}right_link_l" />
           <child link="${prefix}right_link_e" />
@@ -426,5 +426,5 @@
           <limit lower="-1.745" upper="1.745" effort="0" velocity="2.62" />
     </joint>
-    <joint name="${prefix}right_joint_e" type="revolute">
+    <joint name="${prefix}right_joint_3_e" type="revolute">
           <parent link="${prefix}right_link_e" />
           <child link="${prefix}right_link_u" />
@@ -433,5 +433,5 @@
           <limit lower="-2.966" upper="2.966" effort="0" velocity="2.97" />
     </joint>
-    <joint name="${prefix}right_joint_u" type="revolute">
+    <joint name="${prefix}right_joint_4_u" type="revolute">
           <parent link="${prefix}right_link_u" />
           <child link="${prefix}right_link_r" />
@@ -440,5 +440,5 @@
           <limit lower="-1.396" upper="0.7504" effort="0" velocity="2.97" />
     </joint>
-    <joint name="${prefix}right_joint_r" type="revolute">
+    <joint name="${prefix}right_joint_5_r" type="revolute">
           <parent link="${prefix}right_link_r" />
           <child link="${prefix}right_link_b" />
@@ -447,5 +447,5 @@
           <limit lower="-3.1415" upper="3.1415" effort="0" velocity="3.49" />
     </joint>
-    <joint name="${prefix}right_joint_b" type="revolute">
+    <joint name="${prefix}right_joint_6_b" type="revolute">
           <parent link="${prefix}right_link_b" />
           <child link="${prefix}right_link_t" />
@@ -454,5 +454,5 @@
           <limit lower="-1.9198" upper="1.9198" effort="0" velocity="3.49" />
     </joint>
-    <joint name="${prefix}right_joint_t" type="revolute">
+    <joint name="${prefix}right_joint_7_t" type="revolute">
           <parent link="${prefix}right_link_t" />
           <child link="${prefix}right_tool0" />
@@ -469,5 +469,5 @@
           <limit lower="-3.1415" upper="3.1415" effort="0" velocity="2.27" />
     </joint>
-    <joint name="${prefix}left_joint_s" type="revolute">
+    <joint name="${prefix}left_joint_1_s" type="revolute">
           <parent link="${prefix}torso_link_b1" />
           <child link="${prefix}left_link_l" />
@@ -476,5 +476,5 @@
           <limit lower="-1.570" upper="3.1415" effort="0" velocity="2.97" />
     </joint>
-    <joint name="${prefix}left_joint_l" type="revolute">
+    <joint name="${prefix}left_joint_2_l" type="revolute">
           <parent link="${prefix}left_link_l" />
           <child link="${prefix}left_link_e" />
@@ -483,5 +483,5 @@
           <limit lower="-1.745" upper="1.745" effort="0" velocity="2.62" />
     </joint>
-    <joint name="${prefix}left_joint_e" type="revolute">
+    <joint name="${prefix}left_joint_3_e" type="revolute">
           <parent link="${prefix}left_link_e" />
           <child link="${prefix}left_link_u" />
@@ -490,5 +490,5 @@
         <limit lower="-2.966" upper="2.966" effort="0" velocity="2.97" />
     </joint>
-    <joint name="${prefix}left_joint_u" type="revolute">
+    <joint name="${prefix}left_joint_4_u" type="revolute">
           <parent link="${prefix}left_link_u" />
           <child link="${prefix}left_link_r" />
@@ -497,5 +497,5 @@
           <limit lower="-1.396" upper="0.7504" effort="0" velocity="2.97" />
     </joint>
-    <joint name="${prefix}left_joint_r" type="revolute">
+    <joint name="${prefix}left_joint_5_r" type="revolute">
           <parent link="${prefix}left_link_r" />
           <child link="${prefix}left_link_b" />
@@ -504,5 +504,5 @@
           <limit lower="-3.1415" upper="3.1415" effort="0" velocity="3.49" />
     </joint>
-    <joint name="${prefix}left_joint_b" type="revolute">
+    <joint name="${prefix}left_joint_6_b" type="revolute">
           <parent link="${prefix}left_link_b" />
           <child link="${prefix}left_link_t" />
@@ -511,5 +511,5 @@
           <limit lower="-1.9198" upper="1.9198" effort="0" velocity="3.49" />
     </joint>
-     <joint name="${prefix}left_joint_t" type="revolute">
+     <joint name="${prefix}left_joint_7_t" type="revolute">
           <parent link="${prefix}left_link_t" />
           <child link="${prefix}left_tool0" />
