Commit message: Reduce limits for joint u to avoid collisions.

File: motoman_mh6_support/urdf/mh6.urdf (robot description, URDF)
Before this commit: robot motoman_mh6, 7 links, 6 joints
Joints:
- joint joint_u: limit lower=-3.05432619099 upper=4.36332312999 effort=100 velocity=3.83972435439 -> lower=-1.57079632679 upper=3.14159265359 effort=100 velocity=3.83972435439

File: motoman_mh6_support/urdf/mh6_macro.xacro (robot description, xacro)
@@ -129,6 +129,7 @@
 			<origin xyz="0 0 0.614" />
 			<axis xyz="0 -1 0" />
-			<!-- These limits are from the datasheet, but they always cause self collisions. -->
-			<limit lower="${-175 * pi / 180}" upper="${250 * pi / 180}" effort="100" velocity="${220 * pi / 180}" />
+			<!-- These limits are smaller than the datasheet, but the datasheet limits are in collision. -->
+			<!-- Datasheet says [-175, 250] degrees. -->
+			<limit lower="${-90 * pi / 180}" upper="${pi}" effort="100" velocity="${220 * pi / 180}" />
 		</joint>
 		<joint name="${prefix}joint_r" type="revolute">
