Commit message: Updates to CMakeLists and package.xml; --inorder tag added to xacro load

File: motoman_es165rdii_support/urdf/es165rdii_macro.xacro (robot description, xacro)
@@ -143,5 +143,5 @@
                     <mesh filename="package://motoman_es165rdii_support/meshes/es165rdii/visual/balancer_rod.stl"/>
                 </geometry>
-                <material name="${prefix}black">
+                <material name="${prefix}blue">
                     <color rgba="1 1 1 1"/>
                 </material>
@@ -152,5 +152,5 @@
                     <mesh filename="package://motoman_es165rdii_support/meshes/es165rdii/collision/balancer_rod.stl"/>
                 </geometry>
-                <material name="${prefix}black"/>
+                <material name="${prefix}yellow"/>
             </collision>
         </link>
