Commit message: Initial commit for ES200RN-120 support

File: motoman_es_support/urdf/es200rn_120_macro.xacro (robot description, xacro)
@@ -1,15 +1,15 @@
 <?xml version="1.0"?>
 <robot xmlns:xacro="http://ros.org/wiki/xacro">
-  <xacro:macro name="motoman_es165rdii" params="prefix">
+  <xacro:macro name="motoman_es200rn_120" params="prefix">
     <!-- link list -->
     <link name="${prefix}base_link">
       <visual>
         <origin xyz="0 0 0" rpy="0 0 0"/>
-          <geometry>
-            <mesh filename="package://motoman_es_support/meshes/es/visual/base_link.stl"/>
-          </geometry>
-          <material name="blue">
-            <color rgba="0 0 1 1"/>
-          </material>
+        <geometry>
+          <mesh filename="package://motoman_es_support/meshes/es/visual/base_link.stl"/>
+        </geometry>
+        <material name="blue">
+          <color rgba="0 0 1 1"/>
+        </material>
       </visual>
       <collision>
@@ -58,12 +58,12 @@
         <origin xyz="0 0 0" rpy="0 0 0"/>
         <geometry>
-          <mesh filename="package://motoman_es_support/meshes/es165rdii/visual/link_u.stl"/>
-        </geometry>
-        <material name="blue"/>
-      </visual>
-      <collision>
-        <origin xyz="0 0 0" rpy="0 0 0"/>
-        <geometry>
-          <mesh filename="package://motoman_es_support/meshes/es165rdii/collision/link_u.stl"/>
+          <mesh filename="package://motoman_es_support/meshes/es200rn_120/visual/link_u.stl"/>
+        </geometry>
+        <material name="blue"/>
+      </visual>
+      <collision>
+        <origin xyz="0 0 0" rpy="0 0 0"/>
+        <geometry>
+          <mesh filename="package://motoman_es_support/meshes/es200rn_120/collision/link_u.stl"/>
         </geometry>
         <material name="yellow"/>
@@ -73,13 +73,13 @@
       <visual>
         <origin xyz="0 0 0" rpy="0 0 0"/>
-      <geometry>
-        <mesh filename="package://motoman_es_support/meshes/es165rdii/visual/link_r.stl"/>
-      </geometry>
-      <material name="blue"/>
-      </visual>
-      <collision>
-        <origin xyz="0 0 0" rpy="0 0 0"/>
-        <geometry>
-          <mesh filename="package://motoman_es_support/meshes/es165rdii/collision/link_r.stl"/>
+        <geometry>
+          <mesh filename="package://motoman_es_support/meshes/es200rn_120/visual/link_r.stl"/>
+        </geometry>
+        <material name="blue"/>
+      </visual>
+      <collision>
+        <origin xyz="0 0 0" rpy="0 0 0"/>
+        <geometry>
+          <mesh filename="package://motoman_es_support/meshes/es200rn_120/collision/link_r.stl"/>
         </geometry>
         <material name="yellow"/>
@@ -105,10 +105,10 @@
       <visual>
         <origin xyz="0 0 0" rpy="0 0 0"/>
-          <geometry>
-            <mesh filename="package://motoman_es_support/meshes/es/visual/link_t.stl"/>
-          </geometry>
-          <material name="black">
-            <color rgba="0 0 0 1"/>
-          </material>
+        <geometry>
+          <mesh filename="package://motoman_es_support/meshes/es/visual/link_t.stl"/>
+        </geometry>
+        <material name="black">
+          <color rgba="0 0 0 1"/>
+        </material>
       </visual>
       <collision>
@@ -143,7 +143,5 @@
           <mesh filename="package://motoman_es_support/meshes/es/visual/balancer_rod.stl"/>
         </geometry>
-        <material name="blue">
-          <color rgba="1 1 1 1"/>
-        </material>
+        <material name="blue"/>
       </visual>
       <collision>
@@ -162,5 +160,5 @@
       <child link="${prefix}link_s"/>
       <axis xyz="0 0 1"/>
-      <limit lower="${-radians(180)}" upper="${radians(180)}" effort="0" velocity="${radians(105)}"/>
+      <limit lower="${radians(-180)}" upper="${radians(180)}" effort="0" velocity="${radians(90)}"/>
     </joint>
     <joint name="${prefix}joint_2" type="revolute">
@@ -169,5 +167,5 @@
       <child link="${prefix}link_l"/>
       <axis xyz="0 1 0"/>
-      <limit lower="${-radians(130)}" upper="${radians(80)}" effort="0" velocity="${radians(105)}"/>
+      <limit lower="${radians(-130)}" upper="${radians(80)}" effort="0" velocity="${radians(85)}"/>
     </joint>
     <joint name="${prefix}joint_3" type="revolute">
@@ -176,5 +174,5 @@
       <child link="${prefix}link_u"/>
       <axis xyz="0 1 0"/>
-      <limit lower="${-radians(180)}" upper="${radians(79.4)}" effort="0" velocity="${radians(105)}"/>
+      <limit lower="${radians(-180)}" upper="${radians(79.4)}" effort="0" velocity="${radians(85)}"/>
     </joint>
     <joint name="${prefix}joint_4" type="revolute">
@@ -183,12 +181,12 @@
       <child link="${prefix}link_r"/>
       <axis xyz="0 0 -1"/>
-      <limit lower="${-radians(360)}" upper="${radians(360)}" effort="0" velocity="${radians(175)}"/>
+      <limit lower="${radians(-360)}" upper="${radians(360)}" effort="0" velocity="${radians(175)}"/>
     </joint>
     <joint name="${prefix}joint_5" type="revolute">
-      <origin xyz="0 0 -1.225" rpy="0 0 0"/>
+      <origin xyz="0 0 -2.100" rpy="0 0 0"/>
       <parent link="${prefix}link_r"/>
       <child link="${prefix}link_b"/>
       <axis xyz="0 1 0"/>
-      <limit lower="${-radians(130)}" upper="${radians(130)}" effort="0" velocity="${radians(150)}"/>
+      <limit lower="${radians(-130)}" upper="${radians(130)}" effort="0" velocity="${radians(145)}"/>
     </joint>
     <joint name="${prefix}joint_6" type="revolute">
@@ -197,8 +195,8 @@
       <child link="${prefix}link_t"/>
       <axis xyz="0 0 -1"/>
-      <limit lower="${-radians(360)}" upper="${radians(360)}" effort="0" velocity="${radians(240)}"/>
+      <limit lower="${radians(-360)}" upper="${radians(360)}" effort="0" velocity="${radians(240)}"/>
     </joint>
     <joint name="${prefix}joint_6-tool0" type="fixed">
-      <origin xyz="0 0 0" rpy="0 ${pi} 0"/>
+      <origin xyz="0 0 0" rpy="0 ${radians(180)} 0"/>
       <parent link="${prefix}link_t"/>
       <child link="${prefix}tool0"/>
@@ -216,5 +214,5 @@
     <!-- end of joint list -->
     <!-- ROS base_link to Robot Manufacturer World Coordinates transform -->
-    <link name="${prefix}base" />
+    <link name="${prefix}base"/>
     <joint name="${prefix}base_link-base" type="fixed">
       <origin xyz="0 0 0.450" rpy="0 0 0"/>

Commit message: Various formatting fixes

File: motoman_es_support/urdf/es200rn_120_macro.xacro (robot description, xacro)
@@ -155,5 +155,5 @@
     <!-- end of link list -->
     <!-- joint list -->
-    <joint name="${prefix}joint_1" type="revolute">
+    <joint name="${prefix}joint_s" type="revolute">
       <origin xyz="0 0 0.450" rpy="0 0 0"/>
       <parent link="${prefix}base_link"/>
@@ -162,5 +162,5 @@
       <limit lower="${radians(-180)}" upper="${radians(180)}" effort="0" velocity="${radians(90)}"/>
     </joint>
-    <joint name="${prefix}joint_2" type="revolute">
+    <joint name="${prefix}joint_l" type="revolute">
       <origin xyz="0.740 0 0" rpy="0 0 0"/>
       <parent link="${prefix}link_s"/>
@@ -169,5 +169,5 @@
       <limit lower="${radians(-130)}" upper="${radians(80)}" effort="0" velocity="${radians(85)}"/>
     </joint>
-    <joint name="${prefix}joint_3" type="revolute">
+    <joint name="${prefix}joint_u" type="revolute">
       <origin xyz="1.150 0 0" rpy="0 0 0"/>
       <parent link="${prefix}link_l"/>
@@ -176,5 +176,5 @@
       <limit lower="${radians(-180)}" upper="${radians(79.4)}" effort="0" velocity="${radians(85)}"/>
     </joint>
-    <joint name="${prefix}joint_4" type="revolute">
+    <joint name="${prefix}joint_r" type="revolute">
       <origin xyz="0.250 0 0" rpy="0 0 0"/>
       <parent link="${prefix}link_u"/>
@@ -183,5 +183,5 @@
       <limit lower="${radians(-360)}" upper="${radians(360)}" effort="0" velocity="${radians(175)}"/>
     </joint>
-    <joint name="${prefix}joint_5" type="revolute">
+    <joint name="${prefix}joint_b" type="revolute">
       <origin xyz="0 0 -2.100" rpy="0 0 0"/>
       <parent link="${prefix}link_r"/>
@@ -190,5 +190,5 @@
       <limit lower="${radians(-130)}" upper="${radians(130)}" effort="0" velocity="${radians(145)}"/>
     </joint>
-    <joint name="${prefix}joint_6" type="revolute">
+    <joint name="${prefix}joint_t" type="revolute">
       <origin xyz="0 0 -0.225" rpy="0 0 0"/>
       <parent link="${prefix}link_b"/>
@@ -197,5 +197,5 @@
       <limit lower="${radians(-360)}" upper="${radians(360)}" effort="0" velocity="${radians(240)}"/>
     </joint>
-    <joint name="${prefix}joint_6-tool0" type="fixed">
+    <joint name="${prefix}joint_t-tool0" type="fixed">
       <origin xyz="0 0 0" rpy="0 ${radians(180)} 0"/>
       <parent link="${prefix}link_t"/>

Commit message: Changed joint axis directions to match real robot

File: motoman_es_support/urdf/es200rn_120_macro.xacro (robot description, xacro)
@@ -173,5 +173,5 @@
       <parent link="${prefix}link_l"/>
       <child link="${prefix}link_u"/>
-      <axis xyz="0 1 0"/>
+      <axis xyz="0 -1 0"/>
       <limit lower="${radians(-180)}" upper="${radians(79.4)}" effort="0" velocity="${radians(85)}"/>
     </joint>
@@ -180,5 +180,5 @@
       <parent link="${prefix}link_u"/>
       <child link="${prefix}link_r"/>
-      <axis xyz="0 0 -1"/>
+      <axis xyz="0 0 1"/>
       <limit lower="${radians(-360)}" upper="${radians(360)}" effort="0" velocity="${radians(175)}"/>
     </joint>
@@ -187,5 +187,5 @@
       <parent link="${prefix}link_r"/>
       <child link="${prefix}link_b"/>
-      <axis xyz="0 1 0"/>
+      <axis xyz="0 -1 0"/>
       <limit lower="${radians(-130)}" upper="${radians(130)}" effort="0" velocity="${radians(145)}"/>
     </joint>
@@ -194,5 +194,5 @@
       <parent link="${prefix}link_b"/>
       <child link="${prefix}link_t"/>
-      <axis xyz="0 0 -1"/>
+      <axis xyz="0 0 1"/>
       <limit lower="${radians(-360)}" upper="${radians(360)}" effort="0" velocity="${radians(240)}"/>
     </joint>

Commit message: Modified joint limits to match physical limits; added version0 as argument to driver launch files

File: motoman_es_support/urdf/es200rn_120_macro.xacro (robot description, xacro)
@@ -174,5 +174,5 @@
       <child link="${prefix}link_u"/>
       <axis xyz="0 -1 0"/>
-      <limit lower="${radians(-180)}" upper="${radians(79.4)}" effort="0" velocity="${radians(85)}"/>
+      <limit lower="${radians(-138.0)}" upper="${radians(78.0)}" effort="0" velocity="${radians(85)}"/>
     </joint>
     <joint name="${prefix}joint_r" type="revolute">
