Commit message: Base frame relocated per Motoman standard; datasheet URL in package.xml; robot interface launch file renamed

File: motoman_es_support/urdf/es165rdii_macro.xacro (robot description, xacro)
@@ -218,5 +218,5 @@
     <link name="${prefix}base" />
     <joint name="${prefix}base_link-base" type="fixed">
-      <origin xyz="0 0 0" rpy="0 0 0"/>
+      <origin xyz="0 0 0.450" rpy="0 0 0"/>
       <parent link="${prefix}base_link"/>
       <child link="${prefix}base"/>

Commit message: Minor formatting changes

File: motoman_es_support/urdf/es165rdii_macro.xacro (robot description, xacro)
@@ -157,5 +157,5 @@
     <!-- end of link list -->
     <!-- joint list -->
-    <joint name="${prefix}joint_1" type="revolute">
+    <joint name="${prefix}joint_s" type="revolute">
       <origin xyz="0 0 0.450" rpy="0 0 0"/>
       <parent link="${prefix}base_link"/>
@@ -164,5 +164,5 @@
       <limit lower="${-radians(180)}" upper="${radians(180)}" effort="0" velocity="${radians(105)}"/>
     </joint>
-    <joint name="${prefix}joint_2" type="revolute">
+    <joint name="${prefix}joint_l" type="revolute">
       <origin xyz="0.740 0 0" rpy="0 0 0"/>
       <parent link="${prefix}link_s"/>
@@ -171,5 +171,5 @@
       <limit lower="${-radians(130)}" upper="${radians(80)}" effort="0" velocity="${radians(105)}"/>
     </joint>
-    <joint name="${prefix}joint_3" type="revolute">
+    <joint name="${prefix}joint_u" type="revolute">
       <origin xyz="1.150 0 0" rpy="0 0 0"/>
       <parent link="${prefix}link_l"/>
@@ -178,5 +178,5 @@
       <limit lower="${-radians(180)}" upper="${radians(79.4)}" effort="0" velocity="${radians(105)}"/>
     </joint>
-    <joint name="${prefix}joint_4" type="revolute">
+    <joint name="${prefix}joint_r" type="revolute">
       <origin xyz="0.250 0 0" rpy="0 0 0"/>
       <parent link="${prefix}link_u"/>
@@ -185,5 +185,5 @@
       <limit lower="${-radians(360)}" upper="${radians(360)}" effort="0" velocity="${radians(175)}"/>
     </joint>
-    <joint name="${prefix}joint_5" type="revolute">
+    <joint name="${prefix}joint_b" type="revolute">
       <origin xyz="0 0 -1.225" rpy="0 0 0"/>
       <parent link="${prefix}link_r"/>
@@ -192,5 +192,5 @@
       <limit lower="${-radians(130)}" upper="${radians(130)}" effort="0" velocity="${radians(150)}"/>
     </joint>
-    <joint name="${prefix}joint_6" type="revolute">
+    <joint name="${prefix}joint_t" type="revolute">
       <origin xyz="0 0 -0.225" rpy="0 0 0"/>
       <parent link="${prefix}link_b"/>
@@ -199,5 +199,5 @@
       <limit lower="${-radians(360)}" upper="${radians(360)}" effort="0" velocity="${radians(240)}"/>
     </joint>
-    <joint name="${prefix}joint_6-tool0" type="fixed">
+    <joint name="${prefix}joint_t-tool0" type="fixed">
       <origin xyz="0 0 0" rpy="0 ${pi} 0"/>
       <parent link="${prefix}link_t"/>

Commit message: Modified joint limits to reflect extended physical limits

File: motoman_es_support/urdf/es165rdii_macro.xacro (robot description, xacro)
@@ -175,6 +175,6 @@
       <parent link="${prefix}link_l"/>
       <child link="${prefix}link_u"/>
-      <axis xyz="0 1 0"/>
-      <limit lower="${-radians(180)}" upper="${radians(79.4)}" effort="0" velocity="${radians(105)}"/>
+      <axis xyz="0 -1 0"/>
+      <limit lower="${-radians(138.0)}" upper="${radians(78.0)}" effort="0" velocity="${radians(105)}"/>
     </joint>
     <joint name="${prefix}joint_r" type="revolute">
@@ -182,5 +182,5 @@
       <parent link="${prefix}link_u"/>
       <child link="${prefix}link_r"/>
-      <axis xyz="0 0 -1"/>
+      <axis xyz="0 0 1"/>
       <limit lower="${-radians(360)}" upper="${radians(360)}" effort="0" velocity="${radians(175)}"/>
     </joint>
@@ -189,5 +189,5 @@
       <parent link="${prefix}link_r"/>
       <child link="${prefix}link_b"/>
-      <axis xyz="0 1 0"/>
+      <axis xyz="0 -1 0"/>
       <limit lower="${-radians(130)}" upper="${radians(130)}" effort="0" velocity="${radians(150)}"/>
     </joint>
@@ -196,5 +196,5 @@
       <parent link="${prefix}link_b"/>
       <child link="${prefix}link_t"/>
-      <axis xyz="0 0 -1"/>
+      <axis xyz="0 0 1"/>
       <limit lower="${-radians(360)}" upper="${radians(360)}" effort="0" velocity="${radians(240)}"/>
     </joint>

Commit message: es165: use 'correct' joint names.
See ros-industrial/motoman#53.

File: motoman_es_support/urdf/es165rdii_macro.xacro (robot description, xacro)
@@ -157,5 +157,5 @@
     <!-- end of link list -->
     <!-- joint list -->
-    <joint name="${prefix}joint_s" type="revolute">
+    <joint name="${prefix}joint_1_s" type="revolute">
       <origin xyz="0 0 0.450" rpy="0 0 0"/>
       <parent link="${prefix}base_link"/>
@@ -164,5 +164,5 @@
       <limit lower="${-radians(180)}" upper="${radians(180)}" effort="0" velocity="${radians(105)}"/>
     </joint>
-    <joint name="${prefix}joint_l" type="revolute">
+    <joint name="${prefix}joint_2_l" type="revolute">
       <origin xyz="0.740 0 0" rpy="0 0 0"/>
       <parent link="${prefix}link_s"/>
@@ -171,5 +171,5 @@
       <limit lower="${-radians(130)}" upper="${radians(80)}" effort="0" velocity="${radians(105)}"/>
     </joint>
-    <joint name="${prefix}joint_u" type="revolute">
+    <joint name="${prefix}joint_3_u" type="revolute">
       <origin xyz="1.150 0 0" rpy="0 0 0"/>
       <parent link="${prefix}link_l"/>
@@ -178,5 +178,5 @@
       <limit lower="${-radians(138.0)}" upper="${radians(78.0)}" effort="0" velocity="${radians(105)}"/>
     </joint>
-    <joint name="${prefix}joint_r" type="revolute">
+    <joint name="${prefix}joint_4_r" type="revolute">
       <origin xyz="0.250 0 0" rpy="0 0 0"/>
       <parent link="${prefix}link_u"/>
@@ -185,5 +185,5 @@
       <limit lower="${-radians(360)}" upper="${radians(360)}" effort="0" velocity="${radians(175)}"/>
     </joint>
-    <joint name="${prefix}joint_b" type="revolute">
+    <joint name="${prefix}joint_5_b" type="revolute">
       <origin xyz="0 0 -1.225" rpy="0 0 0"/>
       <parent link="${prefix}link_r"/>
@@ -192,5 +192,5 @@
       <limit lower="${-radians(130)}" upper="${radians(130)}" effort="0" velocity="${radians(150)}"/>
     </joint>
-    <joint name="${prefix}joint_t" type="revolute">
+    <joint name="${prefix}joint_6_t" type="revolute">
       <origin xyz="0 0 -0.225" rpy="0 0 0"/>
       <parent link="${prefix}link_b"/>

Commit message: es165: negative radians(..) argument.
Instead of negating the result of passing a positive limit to radians(..).

File: motoman_es_support/urdf/es165rdii_macro.xacro (robot description, xacro)
@@ -168,5 +168,5 @@
       <child link="${prefix}link_s"/>
       <axis xyz="0 0 1"/>
-      <limit lower="${-radians(180)}" upper="${radians(180)}" effort="0" velocity="${radians(105)}"/>
+      <limit lower="${radians(-180)}" upper="${radians(180)}" effort="0" velocity="${radians(105)}"/>
     </joint>
     <joint name="${prefix}joint_2_l" type="revolute">
@@ -175,5 +175,5 @@
       <child link="${prefix}link_l"/>
       <axis xyz="0 1 0"/>
-      <limit lower="${-radians(130)}" upper="${radians(80)}" effort="0" velocity="${radians(105)}"/>
+      <limit lower="${radians(-130)}" upper="${radians(80)}" effort="0" velocity="${radians(105)}"/>
     </joint>
     <joint name="${prefix}joint_3_u" type="revolute">
@@ -182,5 +182,5 @@
       <child link="${prefix}link_u"/>
       <axis xyz="0 -1 0"/>
-      <limit lower="${-radians(138.0)}" upper="${radians(78.0)}" effort="0" velocity="${radians(105)}"/>
+      <limit lower="${radians(-138.0)}" upper="${radians(78.0)}" effort="0" velocity="${radians(105)}"/>
     </joint>
     <joint name="${prefix}joint_4_r" type="revolute">
@@ -189,5 +189,5 @@
       <child link="${prefix}link_r"/>
       <axis xyz="0 0 1"/>
-      <limit lower="${-radians(360)}" upper="${radians(360)}" effort="0" velocity="${radians(175)}"/>
+      <limit lower="${radians(-360)}" upper="${radians(360)}" effort="0" velocity="${radians(175)}"/>
     </joint>
     <joint name="${prefix}joint_5_b" type="revolute">
@@ -196,5 +196,5 @@
       <child link="${prefix}link_b"/>
       <axis xyz="0 -1 0"/>
-      <limit lower="${-radians(130)}" upper="${radians(130)}" effort="0" velocity="${radians(150)}"/>
+      <limit lower="${radians(-130)}" upper="${radians(130)}" effort="0" velocity="${radians(150)}"/>
     </joint>
     <joint name="${prefix}joint_6_t" type="revolute">
@@ -203,5 +203,5 @@
       <child link="${prefix}link_t"/>
       <axis xyz="0 0 1"/>
-      <limit lower="${-radians(360)}" upper="${radians(360)}" effort="0" velocity="${radians(240)}"/>
+      <limit lower="${radians(-360)}" upper="${radians(360)}" effort="0" velocity="${radians(240)}"/>
     </joint>
     <joint name="${prefix}joint_t-tool0" type="fixed">

Commit message: es165: joint U limit according to current specs.

File: motoman_es_support/urdf/es165rdii_macro.xacro (robot description, xacro)
@@ -182,5 +182,5 @@
       <child link="${prefix}link_u"/>
       <axis xyz="0 -1 0"/>
-      <limit lower="${radians(-138.0)}" upper="${radians(78.0)}" effort="0" velocity="${radians(105)}"/>
+      <limit lower="${radians(-112)}" upper="${radians(208)}" effort="0" velocity="${radians(105)}"/>
     </joint>
     <joint name="${prefix}joint_4_r" type="revolute">
