Commit message: URDF correction, code clean up and bug fixing

File: motoman_csda10f_support/urdf/arm_macro.xacro (robot description, xacro)
@@ -166,5 +166,5 @@
 		</joint>
     <joint name="${prefix}joint_tool0" type="fixed" >
-      <origin xyz="0 0 0.0" rpy="3.13 0 0"/>
+      <origin xyz="0 0 -0.057" rpy="3.13 0 0"/>
       <parent link="${prefix}link_7_t" />
       <child link="${prefix}link_tool0" />

File: motoman_csda10f_support/urdf/csda10f_macro.xacro (robot description, xacro)
@@ -1,13 +1,19 @@
 <?xml version="1.0" ?>
-<robot xmlns:xacro="http://ros.org/wiki/xacro"
-    name="csda10f">
+<robot xmlns:xacro="http://ros.org/wiki/xacro">
+        <!--Import torso and arm macros-->
         <xacro:include filename="$(find motoman_csda10f_support)/urdf/common_torso_macro.xacro" />
         <xacro:include filename="$(find motoman_csda10f_support)/urdf/arm_macro.xacro" />
-        <xacro:torso name="torso" prefix="torso_"/>
-        <xacro:motoman_arm name="arm_left" prefix="arm_left_" parent="torso_link_b1" reflect="1">
-            <origin xyz="0.1 0.023 0.3381" rpy="1.57 0 0" />
-        </xacro:motoman_arm>
-        <xacro:motoman_arm name="arm_right" prefix="arm_right_" parent="torso_link_b1" reflect="-1">
-            <origin xyz="0.1 -0.023 0.3381" rpy="1.57 0 0" />
-        </xacro:motoman_arm>
+        <!--Robot instance-->
+        <xacro:macro name="motoman_csda10f" params="prefix">
+            <!--Torso instance-->
+            <xacro:torso name="torso" prefix="torso_"/>
+            <!--Arm instance joint parameters-->
+            <xacro:motoman_arm name="arm_left" prefix="arm_left_" parent="torso_link_b1" reflect="1">
+                <origin xyz="0.1 0.023 0.3381" rpy="1.57 0 0" />
+            </xacro:motoman_arm>
+            <!--Arm instance joint parameters-->
+            <xacro:motoman_arm name="arm_right" prefix="arm_right_" parent="torso_link_b1" reflect="-1">
+                <origin xyz="0.1 -0.023 0.3381" rpy="1.57 0 0" />
+            </xacro:motoman_arm>
+        </xacro:macro>
 </robot>

Commit message: Update arm_macro.xacro
Update the position of tool_0

File: motoman_csda10f_support/urdf/arm_macro.xacro (robot description, xacro)
@@ -166,5 +166,5 @@
 		</joint>
     <joint name="${prefix}joint_tool0" type="fixed" >
-      <origin xyz="0 0 -0.057" rpy="3.13 0 0"/>
+      <origin xyz="0 0 -0.059427" rpy="3.13 0 0"/>
       <parent link="${prefix}link_7_t" />
       <child link="${prefix}link_tool0" />

Commit message: Correction of tool 0 on robot flange: Cordinate frame was misplaced before

File: motoman_csda10f_support/urdf/arm_macro.xacro (robot description, xacro)
@@ -166,5 +166,5 @@
 		</joint>
     <joint name="${prefix}joint_tool0" type="fixed" >
-      <origin xyz="0 0 -0.057" rpy="3.13 0 0"/>
+      <origin xyz="0 0 -0.0569999" rpy="3.13 0 0"/>
       <parent link="${prefix}link_7_t" />
       <child link="${prefix}link_tool0" />

Commit message: Fix arm macro: joint T axis direction was incorrectly oriented

File: motoman_csda10f_support/urdf/arm_macro.xacro (robot description, xacro)
@@ -162,5 +162,5 @@
 			<child link="${prefix}link_7_t"/>
 			<origin xyz="0 0.118 -0.015" rpy="1.57 0 0"/>
-			<axis xyz="0 0 ${-reflect}" />
+			<axis xyz="0 0 ${reflect}" />
 			<limit lower="-3.13" upper="3.13" effort="0" velocity="6.97" />
 		</joint>

Commit message: Correct CSDA10F arm link joints to avoid controller joint limit alarm

File: motoman_csda10f_support/urdf/arm_macro.xacro (robot description, xacro)
@@ -121,5 +121,5 @@
 			<origin xyz="0.1 ${reflect*0.023} 0.3381" rpy="1.57 0 ${(reflect-1)*1.57}"/>
 			<axis xyz="0 0 ${-reflect}" />
-			<limit lower="-3.13" upper="3.13" effort="0" velocity="2.95" />
+			<limit lower="-2.95" upper="2.95" effort="0" velocity="2.95" />
 		</joint>
 		<joint name="${prefix}joint_2_l" type="revolute">
@@ -142,5 +142,5 @@
 			<origin xyz="0.00001 -0.0155 -0.185" rpy="-1.57 0 0"/>
 			<axis xyz="0 0 ${reflect}" />
-			<limit lower="-2.36" upper="2.36" effort="0" velocity="2.95" />
+			<limit lower="-2.35" upper="2.35" effort="0" velocity="2.95" />
 		</joint>
 		<joint name="${prefix}joint_5_r" type="revolute">
