Commit message: corrected property element

File: motoman_gp180_120_support/urdf/gp180_120_macro.xacro (robot description, xacro)
@@ -6,5 +6,5 @@
           <color rgba="0.12941 0.14902 0.74902 1" />
     </material>
-    <xacro:property name="DEG2RAD" value="0.017453292519943295" />
+    <property name="DEG2RAD" value="0.017453292519943295" />
     <!-- link list -->
     <link name="${prefix}base_link">
@@ -171,4 +171,4 @@
         <child link="${prefix}base"/>
     </joint>
-    </xacro:macro>
+</xacro:macro>
 </robot>
