Commit message: mhj: indent two spaces per level.
And convert tabs->spaces.

File: motoman_mhj_support/urdf/mhj.xacro (robot description, xacro)
@@ -1,5 +1,5 @@
 <?xml version="1.0" ?>
 <robot name="motoman_mhj" xmlns:xacro="http://ros.org/wiki/xacro">
-	<xacro:include filename="$(find motoman_mhj_support)/urdf/mhj_macro.xacro" />
-	<xacro:motoman_mhj prefix=""/>
+  <xacro:include filename="$(find motoman_mhj_support)/urdf/mhj_macro.xacro" />
+  <xacro:motoman_mhj prefix=""/>
 </robot>

File: motoman_mhj_support/urdf/mhj_macro.xacro (robot description, xacro)
@@ -1,5 +1,5 @@
 <?xml version="1.0" ?>
 <robot xmlns:xacro="http://ros.org/wiki/xacro">
-<xacro:macro name="motoman_mhj" params="prefix">
+  <xacro:macro name="motoman_mhj" params="prefix">
     <!-- Properties -->
     <material name="yaskawa_blue">
@@ -156,4 +156,4 @@
         <child link="${prefix}base"/>
     </joint>
-    </xacro:macro>
+  </xacro:macro>
 </robot>
