Commit message: Changed color to white
Changed color to white

File: motoman_mhj_support/urdf/mhj_macro.xacro (robot description, xacro)
@@ -3,6 +3,6 @@
   <xacro:macro name="motoman_mhj" params="prefix">
     <!-- Properties -->
-    <material name="yaskawa_blue">
-          <color rgba="0.12941 0.14902 0.74902 1" />
+    <material name="yaskawa_white">
+          <color rgba="0.99 0.99 0.99 1" />
     </material>
     <!-- link list -->
@@ -12,5 +12,5 @@
                 <mesh filename="package://motoman_mhj_support/meshes/mhj/visual/base_link.stl"/>
             </geometry>
-            <material name="yaskawa_blue"/>
+            <material name="yaskawa_white"/>
         </visual>
         <collision>
@@ -25,5 +25,5 @@
                 <mesh filename="package://motoman_mhj_support/meshes/mhj/visual/link_1_s.stl"/>
             </geometry>
-            <material name="yaskawa_blue"/>
+            <material name="yaskawa_white"/>
         </visual>
         <collision>
@@ -38,5 +38,5 @@
                 <mesh filename="package://motoman_mhj_support/meshes/mhj/visual/link_2_l.stl"/>
             </geometry>
-            <material name="yaskawa_blue"/>
+            <material name="yaskawa_white"/>
         </visual>
         <collision>
@@ -51,5 +51,5 @@
                 <mesh filename="package://motoman_mhj_support/meshes/mhj/visual/link_3_u.stl"/>
             </geometry>
-            <material name="yaskawa_blue"/>
+            <material name="yaskawa_white"/>
         </visual>
         <collision>
@@ -64,5 +64,5 @@
                 <mesh filename="package://motoman_mhj_support/meshes/mhj/visual/link_4_r.stl"/>
             </geometry>
-            <material name="yaskawa_blue"/>
+            <material name="yaskawa_white"/>
         </visual>
         <collision>
@@ -77,5 +77,5 @@
                 <mesh filename="package://motoman_mhj_support/meshes/mhj/visual/link_5_b.stl"/>
             </geometry>
-            <material name="yaskawa_blue"/>
+            <material name="yaskawa_white"/>
         </visual>
         <collision>
@@ -90,5 +90,5 @@
                 <mesh filename="package://motoman_mhj_support/meshes/mhj/visual/link_6_t.stl"/>
             </geometry>
-            <material name="yaskawa_blue"/>
+            <material name="yaskawa_white"/>
         </visual>
         <collision>
