Commit message: Updated mh180 based on testing with the real thing. Flipped rotational axis for 3-6 and changed the limit of 3

File: motoman_mh_support/urdf/mh180_120_macro.xacro (robot description, xacro)
@@ -141,6 +141,6 @@
       <parent link="${prefix}link_l"/>
       <child link="${prefix}link_u"/>
-      <axis xyz="0 1 0"/>
-      <limit lower="-${radians(142)}" upper="${radians(90)}" effort="0" velocity="${radians(125)}"/>
+      <axis xyz="0 -1 0"/>
+      <limit lower="-${radians(85)}" upper="${radians(90)}" effort="0" velocity="${radians(125)}"/>
     </joint>
     <joint name="${prefix}joint_4" type="revolute">
@@ -148,5 +148,5 @@
       <parent link="${prefix}link_u"/>
       <child link="${prefix}link_r"/>
-      <axis xyz="1 0 0"/>
+      <axis xyz="-1 0 0"/>
       <limit lower="-${radians(360)}" upper="${radians(360)}" effort="0" velocity="${radians(182)}"/>
     </joint>
@@ -155,5 +155,5 @@
       <parent link="${prefix}link_r"/>
       <child link="${prefix}link_b"/>
-      <axis xyz="0 1 0"/>
+      <axis xyz="0 -1 0"/>
       <limit lower="-${radians(130)}" upper="${radians(130)}" effort="0" velocity="${radians(175)}"/>
     </joint>
@@ -162,5 +162,5 @@
       <parent link="${prefix}link_b"/>
       <child link="${prefix}link_t"/>
-      <axis xyz="1 0 0"/>
+      <axis xyz="-1 0 0"/>
       <limit lower="-${radians(360)}" upper="${radians(360)}" effort="0" velocity="${radians(265)}"/>
     </joint>

Commit message: mh: place base meshes in mh180 sub folder.
To clarify they're MH180 base meshes.

File: motoman_mh_support/urdf/mh180_120_macro.xacro (robot description, xacro)
@@ -7,5 +7,5 @@
         <origin xyz="0 0 0" rpy="0 0 0"/>
         <geometry>
-          <mesh filename="package://motoman_mh_support/meshes/mh/visual/base_link.stl"/>
+          <mesh filename="package://motoman_mh_support/meshes/mh180/visual/base_link.stl"/>
         </geometry>
         <material name="blue">
@@ -15,5 +15,5 @@
       <collision>
         <geometry>
-          <mesh filename="package://motoman_mh_support/meshes/mh/collision/base_link.stl"/>
+          <mesh filename="package://motoman_mh_support/meshes/mh180/collision/base_link.stl"/>
         </geometry>
         <material name="yellow">
@@ -26,5 +26,5 @@
         <origin xyz="0 0 0" rpy="0 0 0"/>
         <geometry>
-          <mesh filename="package://motoman_mh_support/meshes/mh/visual/link_s.stl"/>
+          <mesh filename="package://motoman_mh_support/meshes/mh180/visual/link_s.stl"/>
         </geometry>
         <material name="blue"/>
@@ -33,5 +33,5 @@
         <origin xyz="0 0 0" rpy="0 0 0"/>
         <geometry>
-          <mesh filename="package://motoman_mh_support/meshes/mh/collision/link_s.stl"/>
+          <mesh filename="package://motoman_mh_support/meshes/mh180/collision/link_s.stl"/>
         </geometry>
         <material name="yellow"/>
@@ -42,5 +42,5 @@
         <origin xyz="0 0 0" rpy="0 0 0"/>
         <geometry>
-          <mesh filename="package://motoman_mh_support/meshes/mh/visual/link_l.stl"/>
+          <mesh filename="package://motoman_mh_support/meshes/mh180/visual/link_l.stl"/>
         </geometry>
         <material name="blue"/>
@@ -49,5 +49,5 @@
         <origin xyz="0 0 0" rpy="0 0 0"/>
         <geometry>
-          <mesh filename="package://motoman_mh_support/meshes/mh/collision/link_l.stl"/>
+          <mesh filename="package://motoman_mh_support/meshes/mh180/collision/link_l.stl"/>
         </geometry>
         <material name="yellow"/>
@@ -90,5 +90,5 @@
         <origin xyz="0 0 0" rpy="0 0 0"/>
         <geometry>
-          <mesh filename="package://motoman_mh_support/meshes/mh/visual/link_b.stl"/>
+          <mesh filename="package://motoman_mh_support/meshes/mh180/visual/link_b.stl"/>
         </geometry>
         <material name="blue"/>
@@ -97,5 +97,5 @@
         <origin xyz="0 0 0" rpy="0 0 0"/>
         <geometry>
-          <mesh filename="package://motoman_mh_support/meshes/mh/collision/link_b.stl"/>
+          <mesh filename="package://motoman_mh_support/meshes/mh180/collision/link_b.stl"/>
         </geometry>
         <material name="yellow"/>
@@ -106,5 +106,5 @@
         <origin xyz="0 0 0" rpy="0 0 0"/>
         <geometry>
-          <mesh filename="package://motoman_mh_support/meshes/mh/visual/link_t.stl"/>
+          <mesh filename="package://motoman_mh_support/meshes/mh180/visual/link_t.stl"/>
         </geometry>
         <material name="black">
@@ -115,5 +115,5 @@
         <origin xyz="0 0 0" rpy="0 0 0"/>
         <geometry>
-          <mesh filename="package://motoman_mh_support/meshes/mh/collision/link_t.stl"/>
+          <mesh filename="package://motoman_mh_support/meshes/mh180/collision/link_t.stl"/>
         </geometry>
         <material name="black"/>
