Commit message: mh80: fix joint names

File: motoman_mh_support/urdf/mh80_macro.xacro (robot description, xacro)
@@ -122,5 +122,5 @@
   <!-- end of link list -->
   <!-- joint list -->
-  <joint name="${prefix}joint_s" type="revolute">
+  <joint name="${prefix}joint_1_s" type="revolute">
     <origin xyz="0 0 0.540" rpy="0 0 0"/>
     <parent link="${prefix}base_link"/>
@@ -129,5 +129,5 @@
     <limit lower="-3.14159" upper="3.14159" effort="100" velocity="2.967" />
   </joint>
-  <joint name="${prefix}joint_l" type="revolute">
+  <joint name="${prefix}joint_2_l" type="revolute">
     <origin xyz="0.145 0 0" rpy="0 0 0"/>
     <parent link="${prefix}link_s"/>
@@ -136,5 +136,5 @@
     <limit lower="-1.5707" upper="2.3561" effort="100" velocity="2.443" />
   </joint>
-  <joint name="${prefix}joint_u" type="revolute">
+  <joint name="${prefix}joint_3_u" type="revolute">
     <origin xyz="0 0 0.870" rpy="0 0 0"/>
     <parent link="${prefix}link_l"/>
@@ -143,5 +143,5 @@
     <limit lower="-2.9670" upper="4.3807" effort="100" velocity="2.792" />
   </joint>
-  <joint name="${prefix}joint_r" type="revolute">
+  <joint name="${prefix}joint_4_r" type="revolute">
     <origin xyz="0 0 0.210" rpy="0 0 0"/>
     <parent link="${prefix}link_u"/>
@@ -150,5 +150,5 @@
     <limit lower="-6.2831" upper="6.2831" effort="100" velocity="4.014" />
   </joint>
-  <joint name="${prefix}joint_b" type="revolute">
+  <joint name="${prefix}joint_5_b" type="revolute">
     <origin xyz="1.025 0 0" rpy="0 0 0"/>
     <parent link="${prefix}link_r"/>
@@ -157,5 +157,5 @@
     <limit lower="-2.1816" upper="2.1816" effort="100" velocity="4.014" />
   </joint>
-  <joint name="${prefix}joint_t" type="revolute">
+  <joint name="${prefix}joint_6_t" type="revolute">
     <origin xyz="0.175 0 0" rpy="0 0 0"/>
     <parent link="${prefix}link_b"/>

Commit message: mh80: move tool0 link to end of file
All 'special' frames should be defined after the regular links & joints.

File: motoman_mh_support/urdf/mh80_macro.xacro (robot description, xacro)
@@ -119,5 +119,4 @@
     </collision>
   </link>
-  <link name="${prefix}tool0"/>
   <!-- end of link list -->
   <!-- joint list -->
@@ -164,9 +163,4 @@
     <limit lower="-6.2831" upper="6.2831" effort="100" velocity="6.108" />
   </joint>
-  <joint name="${prefix}joint_t-tool0" type="fixed">
-    <origin xyz="0 0 0" rpy="0 0 0"/>
-    <parent link="${prefix}link_t"/>
-    <child link="${prefix}tool0"/>
-  </joint>
   <!-- end of joint list -->
   <!-- ROS base_link to Robot Manufacturer World Coordinates transform -->
@@ -177,4 +171,10 @@
     <child link="${prefix}base"/>
   </joint>
+  <link name="${prefix}tool0"/>
+  <joint name="${prefix}joint_6_t-tool0" type="fixed">
+    <origin xyz="0 0 0" rpy="0 0 0"/>
+    <parent link="${prefix}link_t"/>
+    <child link="${prefix}tool0"/>
+  </joint>
 </xacro:macro>
 </robot>

Commit message: mh80: correct effort limits
Based on data provided by @EricMarcil (https://github.com/ros-industrial/motoman_experimental/pull/52/files#r626926765):

Axis 	Max Acc/Dec Torque[Nm]
1(S) 	4903.32
2(L) 	5883.99
3(U) 	2986.13
4(R) 	772.27
5(B) 	582.52
6(T) 	250.07

File: motoman_mh_support/urdf/mh80_macro.xacro (robot description, xacro)
@@ -126,5 +126,5 @@
     <child link="${prefix}link_s"/>
     <axis xyz="0 0 1"/>
-    <limit lower="-3.14159" upper="3.14159" effort="100" velocity="2.967" />
+    <limit lower="-3.14159" upper="3.14159" effort="4903.32" velocity="2.967" />
   </joint>
   <joint name="${prefix}joint_2_l" type="revolute">
@@ -133,5 +133,5 @@
     <child link="${prefix}link_l"/>
     <axis xyz="0 1 0" />
-    <limit lower="-1.5707" upper="2.3561" effort="100" velocity="2.443" />
+    <limit lower="-1.5707" upper="2.3561" effort="5883.99" velocity="2.443" />
   </joint>
   <joint name="${prefix}joint_3_u" type="revolute">
@@ -140,5 +140,5 @@
     <child link="${prefix}link_u"/>
     <axis xyz="0 -1 0"/>
-    <limit lower="-2.9670" upper="4.3807" effort="100" velocity="2.792" />
+    <limit lower="-2.9670" upper="4.3807" effort="2986.13" velocity="2.792" />
   </joint>
   <joint name="${prefix}joint_4_r" type="revolute">
@@ -147,5 +147,5 @@
     <child link="${prefix}link_r"/>
     <axis xyz="-1 0 0"/>
-    <limit lower="-6.2831" upper="6.2831" effort="100" velocity="4.014" />
+    <limit lower="-6.2831" upper="6.2831" effort="772.27" velocity="4.014" />
   </joint>
   <joint name="${prefix}joint_5_b" type="revolute">
@@ -154,5 +154,5 @@
     <child link="${prefix}link_b"/>
     <axis xyz="0 -1 0" />
-    <limit lower="-2.1816" upper="2.1816" effort="100" velocity="4.014" />
+    <limit lower="-2.1816" upper="2.1816" effort="582.52" velocity="4.014" />
   </joint>
   <joint name="${prefix}joint_6_t" type="revolute">
@@ -161,5 +161,5 @@
     <child link="${prefix}link_t"/>
     <axis xyz="-1 0 0" />
-    <limit lower="-6.2831" upper="6.2831" effort="100" velocity="6.108" />
+    <limit lower="-6.2831" upper="6.2831" effort="250.07" velocity="6.108" />
   </joint>
   <!-- end of joint list -->

Commit message: mh80: use radians(..) everywhere
Instead of manual conversions.

Based on the datasheet linked in the package's manifest (DS-603-D, Jan 2019).

File: motoman_mh_support/urdf/mh80_macro.xacro (robot description, xacro)
@@ -126,5 +126,5 @@
     <child link="${prefix}link_s"/>
     <axis xyz="0 0 1"/>
-    <limit lower="-3.14159" upper="3.14159" effort="4903.32" velocity="2.967" />
+    <limit lower="${radians(-180)}" upper="${radians(180)}" effort="4903.32" velocity="${radians(170)}" />
   </joint>
   <joint name="${prefix}joint_2_l" type="revolute">
@@ -133,5 +133,5 @@
     <child link="${prefix}link_l"/>
     <axis xyz="0 1 0" />
-    <limit lower="-1.5707" upper="2.3561" effort="5883.99" velocity="2.443" />
+    <limit lower="${radians(-90)}" upper="${radians(135)}" effort="5883.99" velocity="${radians(140)}" />
   </joint>
   <joint name="${prefix}joint_3_u" type="revolute">
@@ -140,5 +140,5 @@
     <child link="${prefix}link_u"/>
     <axis xyz="0 -1 0"/>
-    <limit lower="-2.9670" upper="4.3807" effort="2986.13" velocity="2.792" />
+    <limit lower="${radians(-170)}" upper="${radians(251)}" effort="2986.13" velocity="${radians(160)}" />
   </joint>
   <joint name="${prefix}joint_4_r" type="revolute">
@@ -147,5 +147,5 @@
     <child link="${prefix}link_r"/>
     <axis xyz="-1 0 0"/>
-    <limit lower="-6.2831" upper="6.2831" effort="772.27" velocity="4.014" />
+    <limit lower="${radians(-360)}" upper="${radians(360)}" effort="772.27" velocity="${radians(230)}" />
   </joint>
   <joint name="${prefix}joint_5_b" type="revolute">
@@ -154,5 +154,5 @@
     <child link="${prefix}link_b"/>
     <axis xyz="0 -1 0" />
-    <limit lower="-2.1816" upper="2.1816" effort="582.52" velocity="4.014" />
+    <limit lower="${radians(-125)}" upper="${radians(125)}" effort="582.52" velocity="230" />
   </joint>
   <joint name="${prefix}joint_6_t" type="revolute">
@@ -161,5 +161,5 @@
     <child link="${prefix}link_t"/>
     <axis xyz="-1 0 0" />
-    <limit lower="-6.2831" upper="6.2831" effort="250.07" velocity="6.108" />
+    <limit lower="${radians(-360)}" upper="${radians(360)}" effort="250.07" velocity="${radians(350)}" />
   </joint>
   <!-- end of joint list -->

Commit message: mh80: correct tool0 orientation

File: motoman_mh_support/urdf/mh80_macro.xacro (robot description, xacro)
@@ -173,5 +173,5 @@
   <link name="${prefix}tool0"/>
   <joint name="${prefix}joint_6_t-tool0" type="fixed">
-    <origin xyz="0 0 0" rpy="0 0 0"/>
+    <origin xyz="0 0 0" rpy="${radians(180)} ${radians(-90)} 0"/>
     <parent link="${prefix}link_t"/>
     <child link="${prefix}tool0"/>

Commit message: mh80: use material def from resources package

File: motoman_mh_support/urdf/mh80_macro.xacro (robot description, xacro)
@@ -2,4 +2,5 @@
 <robot xmlns:xacro="http://ros.org/wiki/xacro">
 <xacro:macro name="motoman_mh80" params="prefix">
+  <xacro:include filename="$(find motoman_resources)/urdf/common_materials.xacro"/>
   <!-- link list -->
   <link name="${prefix}base_link">
@@ -9,7 +10,5 @@
         <mesh filename="package://motoman_mh_support/meshes/mh80/visual/base_link.stl"/>
       </geometry>
-      <material name="blue">
-        <color rgba="0 0 1 1"/>
-      </material>
+      <xacro:material_yaskawa_blue/>
     </visual>
     <collision>
@@ -18,7 +17,4 @@
         <mesh filename="package://motoman_mh_support/meshes/mh80/collision/base_link.stl"/>
       </geometry>
-      <material name="collision_material">
-        <color rgba="1 0 0 1"/>
-      </material>
     </collision>
   </link>
@@ -29,5 +25,5 @@
         <mesh filename="package://motoman_mh_support/meshes/mh80/visual/link_s.stl"/>
       </geometry>
-      <material name="blue"/>
+      <xacro:material_yaskawa_blue/>
     </visual>
     <collision>
@@ -36,5 +32,4 @@
         <mesh filename="package://motoman_mh_support/meshes/mh80/collision/link_s.stl"/>
       </geometry>
-      <material name="collision_material"/>
     </collision>
   </link>
@@ -45,5 +40,5 @@
         <mesh filename="package://motoman_mh_support/meshes/mh80/visual/link_l.stl"/>
       </geometry>
-      <material name="blue"/>
+      <xacro:material_yaskawa_blue/>
     </visual>
     <collision>
@@ -52,5 +47,4 @@
         <mesh filename="package://motoman_mh_support/meshes/mh80/collision/link_l.stl"/>
       </geometry>
-      <material name="collision_material"/>
     </collision>
   </link>
@@ -61,5 +55,5 @@
         <mesh filename="package://motoman_mh_support/meshes/mh80/visual/link_u.stl"/>
       </geometry>
-      <material name="blue"/>
+      <xacro:material_yaskawa_blue/>
     </visual>
     <collision>
@@ -68,5 +62,4 @@
         <mesh filename="package://motoman_mh_support/meshes/mh80/collision/link_u.stl"/>
       </geometry>
-      <material name="collision_material"/>
     </collision>
   </link>
@@ -77,5 +70,5 @@
         <mesh filename="package://motoman_mh_support/meshes/mh80/visual/link_r.stl"/>
       </geometry>
-      <material name="blue"/>
+      <xacro:material_yaskawa_blue/>
     </visual>
     <collision>
@@ -84,5 +77,4 @@
         <mesh filename="package://motoman_mh_support/meshes/mh80/collision/link_r.stl"/>
       </geometry>
-      <material name="collision_material"/>
     </collision>
   </link>
@@ -93,5 +85,5 @@
         <mesh filename="package://motoman_mh_support/meshes/mh80/visual/link_b.stl"/>
       </geometry>
-      <material name="blue"/>
+      <xacro:material_yaskawa_blue/>
     </visual>
     <collision>
@@ -100,5 +92,4 @@
         <mesh filename="package://motoman_mh_support/meshes/mh80/collision/link_b.stl"/>
       </geometry>
-      <material name="collision_material"/>
     </collision>
   </link>
@@ -109,5 +100,5 @@
         <mesh filename="package://motoman_mh_support/meshes/mh80/visual/link_t.stl"/>
       </geometry>
-      <material name="blue"/>
+      <xacro:material_yaskawa_blue/>
     </visual>
     <collision>
@@ -116,5 +107,4 @@
         <mesh filename="package://motoman_mh_support/meshes/mh80/collision/link_t.stl"/>
       </geometry>
-      <material name="collision_material"/>
     </collision>
   </link>

Commit message: mh80: introduce flange frame
and move the X translation from joint_6_t to the flange joint.

File: motoman_mh_support/urdf/mh80_macro.xacro (robot description, xacro)
@@ -147,5 +147,5 @@
   </joint>
   <joint name="${prefix}joint_6_t" type="revolute">
-    <origin xyz="0.175 0 0" rpy="0 0 0"/>
+    <origin xyz="0 0 0" rpy="0 0 0"/>
     <parent link="${prefix}link_b"/>
     <child link="${prefix}link_t"/>
@@ -161,4 +161,11 @@
     <child link="${prefix}base"/>
   </joint>
+  <!-- ROS-Industrial 'flange' frame: attachment point for EEF models -->
+  <link name="${prefix}flange"/>
+  <joint name="${prefix}joint_6_t-flange" type="fixed">
+    <origin xyz="0.175 0 0" rpy="0 0 0"/>
+    <parent link="${prefix}link_t"/>
+    <child link="${prefix}flange"/>
+  </joint>
   <link name="${prefix}tool0"/>
   <joint name="${prefix}joint_6_t-tool0" type="fixed">

Commit message: mh80: make tool0 child of flange
now that this model has a 'flange' frame.

File: motoman_mh_support/urdf/mh80_macro.xacro (robot description, xacro)
@@ -168,8 +168,9 @@
     <child link="${prefix}flange"/>
   </joint>
+  <!-- ROS-Industrial 'tool0' frame: all-zeros tool frame -->
   <link name="${prefix}tool0"/>
-  <joint name="${prefix}joint_6_t-tool0" type="fixed">
+  <joint name="${prefix}flange-tool0" type="fixed">
     <origin xyz="0 0 0" rpy="${radians(180)} ${radians(-90)} 0"/>
-    <parent link="${prefix}link_t"/>
+    <parent link="${prefix}flange"/>
     <child link="${prefix}tool0"/>
   </joint>
