Commit message: Update motoman_mpx3500_support/urdf/mpx3500_macro.xacro
Co-authored-by: Michael Ripperger <michael.ripperger@swri.org>

File: motoman_mpx3500_support/urdf/mpx3500_macro.xacro (robot description, xacro)
@@ -150,5 +150,5 @@
     </joint>
     <joint name="${prefix}joint_6_t-tool0" type="fixed">
-        <origin xyz="0.123 0 0" rpy="3.1415926 -1.570796 0"/>
+        <origin xyz="0.123 0 0" rpy="${radians(180)} ${radians(-90)} 0"/>
         <parent link="${prefix}link_6_t"/>
         <child link="${prefix}tool0"/>
